File: kicad_hiltop_sensi_board/InputConditioning.sch (KiCad schematic (older format))
At the start: 20 parts, among them U4 AD8646, U5 AD8646

Commit message: Updated LBBC board and Board layout started
Parts:
- U4, U5: footprint (none) -> Package_SO:SOIC-8_3.9x4.9mm_P1.27mm
Changed lines of the file:
@@
 F 0 "U4" H 8519 3346 50  0000 L CNN
 F 1 "AD8646" H 8519 3255 50  0000 L CNN
-F 2 "" H 8175 3300 50  0001 C CNN
+F 2 "Package_SO:SOIC-8_3.9x4.9mm_P1.27mm" H 8175 3300 50  0001 C CNN
 F 3 "" H 8175 3300 50  0001 C CNN
 	2    8175 3300
@@
 F 0 "U4" H 3519 3196 50  0000 L CNN
 F 1 "AD8646" H 3519 3105 50  0000 L CNN
-F 2 "" H 3175 3150 50  0001 C CNN
+F 2 "Package_SO:SOIC-8_3.9x4.9mm_P1.27mm" H 3175 3150 50  0001 C CNN
 F 3 "" H 3175 3150 50  0001 C CNN
 	1    3175 3150
@@
 F 0 "U5" H 8519 5146 50  0000 L CNN
 F 1 "AD8646" H 8519 5055 50  0000 L CNN
-F 2 "" H 8175 5100 50  0001 C CNN
+F 2 "Package_SO:SOIC-8_3.9x4.9mm_P1.27mm" H 8175 5100 50  0001 C CNN
 F 3 "" H 8175 5100 50  0001 C CNN
 	2    8175 5100
@@
 F 0 "U5" H 3519 4996 50  0000 L CNN
 F 1 "AD8646" H 3519 4905 50  0000 L CNN
-F 2 "" H 3175 4950 50  0001 C CNN
+F 2 "Package_SO:SOIC-8_3.9x4.9mm_P1.27mm" H 3175 4950 50  0001 C CNN
 F 3 "" H 3175 4950 50  0001 C CNN
 	1    3175 4950

Commit message: Sensi board updated pin map
Parts:
- C14, C15: footprint Capacitor_SMD:C_0603_1608Metric -> Capacitor_SMD:C_0402_1005Metric
Changed lines of the file:
@@
 F 0 "C14" V 3098 2775 50  0000 C CNN
 F 1 "100nF" V 3189 2775 50  0000 C CNN
-F 2 "Capacitor_SMD:C_0603_1608Metric" H 3388 2625 50  0001 C CNN
+F 2 "Capacitor_SMD:C_0402_1005Metric" H 3388 2625 50  0001 C CNN
 F 3 "" H 3350 2775 50  0001 C CNN
 	1    3350 2775
@@
 F 0 "C15" V 3098 4550 50  0000 C CNN
 F 1 "100nF" V 3189 4550 50  0000 C CNN
-F 2 "Capacitor_SMD:C_0603_1608Metric" H 3388 4400 50  0001 C CNN
+F 2 "Capacitor_SMD:C_0402_1005Metric" H 3388 4400 50  0001 C CNN
 F 3 "" H 3350 4550 50  0001 C CNN
 	1    3350 4550

Commit message: Updated sensi board pin map and layout before PCB tracking
Parts:
- C14, C15: Devtank (none) -> 105-019
- U4, U5: Devtank (none) -> 120-006
Changed lines of the file:
@@
 F 2 "Package_SO:SOIC-8_3.9x4.9mm_P1.27mm" H 8175 3300 50  0001 C CNN
 F 3 "" H 8175 3300 50  0001 C CNN
+F 4 "120-006" H 8175 3300 50  0001 C CNN "Devtank"
 	2    8175 3300
 	1    0    0    -1
@@
 F 2 "Package_SO:SOIC-8_3.9x4.9mm_P1.27mm" H 3175 3150 50  0001 C CNN
 F 3 "" H 3175 3150 50  0001 C CNN
+F 4 "120-006" H 3175 3150 50  0001 C CNN "Devtank"
 	1    3175 3150
 	1    0    0    -1
@@
 F 2 "Package_SO:SOIC-8_3.9x4.9mm_P1.27mm" H 8175 5100 50  0001 C CNN
 F 3 "" H 8175 5100 50  0001 C CNN
+F 4 "120-006" H 8175 5100 50  0001 C CNN "Devtank"
 	2    8175 5100
 	1    0    0    -1
@@
 F 2 "Package_SO:SOIC-8_3.9x4.9mm_P1.27mm" H 3175 4950 50  0001 C CNN
 F 3 "" H 3175 4950 50  0001 C CNN
+F 4 "120-006" H 3175 4950 50  0001 C CNN "Devtank"
 	1    3175 4950
 	1    0    0    -1
@@
 F 2 "Capacitor_SMD:C_0402_1005Metric" H 3388 2625 50  0001 C CNN
 F 3 "" H 3350 2775 50  0001 C CNN
+F 4 "105-019" H 3350 2775 50  0001 C CNN "Devtank"
 	1    3350 2775
 	0    1    1    0
@@
 F 2 "Capacitor_SMD:C_0402_1005Metric" H 3388 4400 50  0001 C CNN
 F 3 "" H 3350 4550 50  0001 C CNN
+F 4 "105-019" H 3350 4550 50  0001 C CNN "Devtank"
 	1    3350 4550
 	0    1    1    0
