File: kicad_hiltop_sensi_board/Temperature.sch (KiCad schematic (older format))
At the start: 21 parts

Commit message: Just about to aad the RTD
Parts:
- C24, C30, C31, C32, C37, C38, C39, C? (x3): symbol device:C -> Sensi_Board-rescue:C-device
- L? (x2): symbol device:Ferrite_Bead -> Sensi_Board-rescue:Ferrite_Bead-device
- R24, R25, R28, R? (x3): symbol device:R -> Sensi_Board-rescue:R-device
- TP? (x2): symbol Connector:Test_Point -> Sensi_Board-rescue:Test_Point-Connector
Changed lines of the file:
@@
 EESchema Schematic File Version 4
 LIBS:Sensi_Board-cache
-EELAYER 29 0
+EELAYER 30 0
 EELAYER END
 $Descr A3 16535 11693
 encoding utf-8
-Sheet 7 8
+Sheet 7 9
 Title "Roving Sensor Design"
 Date "17/10/2017"
@@
 $EndComp
 $Comp
-L device:C C24
+L Sensi_Board-rescue:C-device C24
 U 1 1 59C07C31
 P 9450 2750
@@
 	11950 5100 10800 5100
 $Comp
-L device:C C37
+L Sensi_Board-rescue:C-device C37
 U 1 1 59CBCCB2
 P 8450 2875
@@
 $EndComp
 $Comp
-L device:C C38
+L Sensi_Board-rescue:C-device C38
 U 1 1 59CBD08B
 P 9750 2750
@@
 $EndComp
 $Comp
-L device:C C39
+L Sensi_Board-rescue:C-device C39
 U 1 1 59CBD29F
 P 10750 2550
@@
 $EndComp
 $Comp
-L device:R R28
+L Sensi_Board-rescue:R-device R28
 U 1 1 59CBB35E
 P 8050 7225
@@
 	3850 4750 3850 4850
 $Comp
-L device:R R24
+L Sensi_Board-rescue:R-device R24
 U 1 1 59CBCA4A
 P 3450 4000
@@
 $EndComp
 $Comp
-L device:R R25
+L Sensi_Board-rescue:R-device R25
 U 1 1 59CBCA51
 P 3450 4400
@@
 $EndComp
 $Comp
-L device:C C31
+L Sensi_Board-rescue:C-device C31
 U 1 1 59CBCA58
 P 3850 4200
@@
 $EndComp
 $Comp
-L device:C C30
+L Sensi_Board-rescue:C-device C30
 U 1 1 59CBCA5F
 P 3850 3800
@@
 $EndComp
 $Comp
-L device:C C32
+L Sensi_Board-rescue:C-device C32
 U 1 1 59CBCA66
 P 3850 4600
@@
 	10800 4100 11950 4100
 $Comp
-L Connector:Test_Point TP?
+L Sensi_Board-rescue:Test_Point-Connector TP?
 U 1 1 5D0C65E8
 P 4500 3900
@@
 $EndComp
 $Comp
-L Connector:Test_Point TP?
+L Sensi_Board-rescue:Test_Point-Connector TP?
 U 1 1 5D0C7CF5
 P 4500 4500
@@
 	8300 7225 8550 7225
 $Comp
-L device:R R?
+L Sensi_Board-rescue:R-device R?
 U 1 1 5D20C69A
 P 7900 6700
@@
 	7900 6850 7900 6925
 $Comp
-L device:R R?
+L Sensi_Board-rescue:R-device R?
 U 1 1 5D20C76E
 P 8200 6700
@@
 	8200 6850 8200 6925
 $Comp
-L device:C C?
+L Sensi_Board-rescue:C-device C?
 U 1 1 5D20F734
 P 7675 6350
@@
 $EndComp
 $Comp
-L device:C C?
+L Sensi_Board-rescue:C-device C?
 U 1 1 5D20F92C
 P 8050 6425
@@
 $EndComp
 $Comp
-L device:C C?
+L Sensi_Board-rescue:C-device C?
 U 1 1 5D20F9E3
 P 8425 6350
@@
 	7900 6350 7900 6425
 $Comp
-L device:Ferrite_Bead L?
+L Sensi_Board-rescue:Ferrite_Bead-device L?
 U 1 1 5D238B4F
 P 10350 1950
@@
 	10350 1800 10350 1725
 $Comp
-L device:Ferrite_Bead L?
+L Sensi_Board-rescue:Ferrite_Bead-device L?
 U 1 1 5D2D4852
 P 8850 2200
@@
 	8850 2050 8850 1925
 $Comp
-L device:R R?
+L Sensi_Board-rescue:R-device R?
 U 1 1 5D2C070D
 P 11075 3725
