File: kicad_hiltop_sensi_board/USB_Debug.sch (KiCad schematic (older format))
At the start: 13 parts, among them U13 CP2102N-A01-GQFN24

Commit message: Just about to aad the RTD
Parts:
- C52, C55, C56: symbol device:C -> Sensi_Board-rescue:C-device
- R76, R77, R78, R79, R80, R81, R82, R83, R84: symbol device:R -> Sensi_Board-rescue:R-device
- U13: symbol silabs:CP2102N-A01-GQFN24 -> Sensi_Board-rescue:CP2102N-A01-GQFN24-silabs
Changed lines of the file:
@@
 EESchema Schematic File Version 4
 LIBS:Sensi_Board-cache
-EELAYER 29 0
+EELAYER 30 0
 EELAYER END
 $Descr A4 11693 8268
 encoding utf-8
-Sheet 5 8
+Sheet 4 9
 Title "HILTOP Motherboard"
 Date "2019-01-10"
@@
 USB_N
 $Comp
-L silabs:CP2102N-A01-GQFN24 U13
+L Sensi_Board-rescue:CP2102N-A01-GQFN24-silabs U13
 U 1 1 5C2328D1
 P 5525 3475
@@
 	5525 2325 5525 2450
 $Comp
-L device:R R78
+L Sensi_Board-rescue:R-device R78
 U 1 1 5C3A3F19
 P 4050 3775
@@
 	2675 2875 2975 2875
 $Comp
-L device:R R?
+L Sensi_Board-rescue:R-device R?
 U 1 1 5C3AE29F
 P 6650 3975
@@
 $EndComp
 $Comp
-L device:R R?
+L Sensi_Board-rescue:R-device R?
 U 1 1 5C3AF9C1
 P 6650 4075
@@
 	6125 3275 7125 3275
 $Comp
-L device:R R83
+L Sensi_Board-rescue:R-device R83
 U 1 1 5C3B4D7B
 P 7275 3175
@@
 $EndComp
 $Comp
-L device:R R84
+L Sensi_Board-rescue:R-device R84
 U 1 1 5C3B4EF0
 P 7275 3275
@@
 	7425 3275 7575 3275
 $Comp
-L device:R R76
+L Sensi_Board-rescue:R-device R76
 U 1 1 5C3C0EE1
 P 3125 2875
@@
 $EndComp
 $Comp
-L device:R R77
+L Sensi_Board-rescue:R-device R77
 U 1 1 5C3C0F83
 P 3825 2625
@@
 	3825 2400 3825 2475
 $Comp
-L device:C C55
+L Sensi_Board-rescue:C-device C55
 U 1 1 5C3C60B5
 P 5800 2225
@@
 $EndComp
 $Comp
-L device:C C56
+L Sensi_Board-rescue:C-device C56
 U 1 1 5C3C6FB8
 P 6225 2225
@@
 NoConn ~ 6125 3575
 $Comp
-L device:C C?
+L Sensi_Board-rescue:C-device C?
 U 1 1 5CA83BDF
 P 3475 3275
@@
 	6125 3975 6500 3975
 $Comp
-L device:R R?
+L Sensi_Board-rescue:R-device R?
 U 1 1 5CA8BD2A
 P 6650 3875
@@
 	6125 3875 6500 3875
 $Comp
-L device:R R?
+L Sensi_Board-rescue:R-device R?
 U 1 1 5CA8CA4A
 P 6650 3775

Commit message: updated sensi board for LBBC 04/09/19
Parts:
- added R?: 47K, symbol device:R
- R78: value 0R -> 24K
- R79, R80: value 330R -> 0R
Connections:
- net GND: now also R?.1
- net at R78.1, U13.8 (VBUS): now also R?.2
Changed lines of the file:
@@
 $Descr A4 11693 8268
 encoding utf-8
-Sheet 4 9
+Sheet 4 11
 Title "HILTOP Motherboard"
 Date "2019-01-10"
@@
 P 4050 3775
 F 0 "R78" V 3950 3675 50  0000 C CNN
-F 1 "0R" V 3950 3850 50  0000 C CNN
+F 1 "24K" V 3950 3850 50  0000 C CNN
 F 2 "Resistor_SMD:R_0603_1608Metric" V 3980 3775 50  0001 C CNN
 F 3 "" H 4050 3775 50  0001 C CNN
@@
 $EndComp
 Wire Wire Line
-	4925 3775 4200 3775
+	4925 3775 4300 3775
 Text HLabel 3025 3775 0    60   Input ~ 0
 USB_BUS_PWR
@@
 AR Path="/5CA829FD/5CA8BD2A" Ref="R80"  Part="1"
 F 0 "R80" V 6600 3650 50  0000 C CNN
-F 1 "330R" V 6600 4100 50  0000 C CNN
+F 1 "0R" V 6600 4100 50  0000 C CNN
 F 2 "Resistor_SMD:R_0603_1608Metric" V 6580 3875 50  0001 C CNN
 F 3 "" H 6650 3875 50  0000 C CNN
@@
 AR Path="/5CA829FD/5CA8CA4A" Ref="R79"  Part="1"
 F 0 "R79" V 6600 3550 50  0000 C CNN
-F 1 "330R" V 6600 4000 50  0000 C CNN
+F 1 "0R" V 6600 4000 50  0000 C CNN
 F 2 "Resistor_SMD:R_0603_1608Metric" V 6580 3775 50  0001 C CNN
 F 3 "" H 6650 3775 50  0000 C CNN
@@
 Wire Wire Line
 	4650 2325 4650 3475
+$Comp
+L device:R R?
+U 1 1 605DE563
+P 4300 3550
+F 0 "R?" H 4370 3596 50  0000 L CNN
+F 1 "47K" H 4370 3505 50  0000 L CNN
+F 2 "" V 4230 3550 50  0001 C CNN
+F 3 "" H 4300 3550 50  0001 C CNN
+	1    4300 3550
+	1    0    0    -1
+$EndComp
+$Comp
+L power:GND #PWR?
+U 1 1 605DF18F
+P 4300 3300
+F 0 "#PWR?" H 4300 3050 50  0001 C CNN
+F 1 "GND" H 4305 3127 50  0000 C CNN
+F 2 "" H 4300 3300 50  0001 C CNN
+F 3 "" H 4300 3300 50  0001 C CNN
+	1    4300 3300
+	-1   0    0    1
+$EndComp
+Wire Wire Line
+	4300 3700 4300 3775
+Connection ~ 4300 3775
+Wire Wire Line
+	4300 3775 4200 3775
+Wire Wire Line
+	4300 3300 4300 3400
 $EndSCHEMATC
