File: kicad_hiltop_sensi_board/USB_Debug.sch (KiCad schematic (older format))
At the start: 14 parts, among them U13 CP2102N-A01-GQFN24

Commit message: LBBC sensi board upto date schematic and footprints
Parts:
- R20: footprint (none) -> Resistor_SMD:R_0603_1608Metric
Changed lines of the file:
@@
 $Descr A4 11693 8268
 encoding utf-8
-Sheet 4 11
+Sheet 3 11
 Title "HILTOP Motherboard"
 Date "2019-01-10"
@@
 F 0 "R20" H 4370 3596 50  0000 L CNN
 F 1 "47K" H 4370 3505 50  0000 L CNN
-F 2 "" V 4230 3550 50  0001 C CNN
+F 2 "Resistor_SMD:R_0603_1608Metric" V 4230 3550 50  0001 C CNN
 F 3 "" H 4300 3550 50  0001 C CNN
 	1    4300 3550

Commit message: Sensi board updated pin map
Parts:
- C55: footprint Capacitor_SMD:C_0805_2012Metric -> Capacitor_SMD:C_0402_1005Metric
- C56: footprint Capacitor_SMD:C_0603_1608Metric -> Capacitor_SMD:C_0402_1005Metric
Changed lines of the file:
@@
 F 0 "C55" H 5915 2271 50  0000 L CNN
 F 1 "4.7uF" H 5915 2180 50  0000 L CNN
-F 2 "Capacitor_SMD:C_0805_2012Metric" H 5838 2075 50  0001 C CNN
+F 2 "Capacitor_SMD:C_0402_1005Metric" H 5838 2075 50  0001 C CNN
 F 3 "" H 5800 2225 50  0001 C CNN
 F 4 "105-007" H 5800 2225 50  0001 C CNN "Devtank"
@@
 F 0 "C56" H 6340 2271 50  0000 L CNN
 F 1 "100nF" H 6340 2180 50  0000 L CNN
-F 2 "Capacitor_SMD:C_0603_1608Metric" H 6263 2075 50  0001 C CNN
+F 2 "Capacitor_SMD:C_0402_1005Metric" H 6263 2075 50  0001 C CNN
 F 3 "" H 6225 2225 50  0001 C CNN
 F 4 "105-002" H 6225 2225 50  0001 C CNN "Devtank"

Commit message: Updated sensi board pin map and layout before PCB tracking
Parts:
- C55: Devtank 105-007 -> 105-025
- R20: Devtank (none) -> 101-016
- R78: Devtank 101-005 -> 101-055
- R79, R80: Devtank 101-024 -> 101-005
Changed lines of the file:
@@
 F 2 "Resistor_SMD:R_0603_1608Metric" V 3980 3775 50  0001 C CNN
 F 3 "" H 4050 3775 50  0001 C CNN
-F 4 "101-005" V 4050 3775 50  0001 C CNN "Devtank"
+F 4 "101-055" V 4050 3775 50  0001 C CNN "Devtank"
 	1    4050 3775
 	0    1    1    0
@@
 F 2 "Capacitor_SMD:C_0402_1005Metric" H 5838 2075 50  0001 C CNN
 F 3 "" H 5800 2225 50  0001 C CNN
-F 4 "105-007" H 5800 2225 50  0001 C CNN "Devtank"
+F 4 "105-025" H 5800 2225 50  0001 C CNN "Devtank"
 	1    5800 2225
 	1    0    0    -1
@@
 F 2 "Resistor_SMD:R_0603_1608Metric" V 6580 3875 50  0001 C CNN
 F 3 "" H 6650 3875 50  0000 C CNN
-F 4 "101-024" V 6650 3875 60  0001 C CNN "Devtank"
+F 4 "101-005" V 6650 3875 60  0001 C CNN "Devtank"
 	1    6650 3875
 	0    1    1    0
@@
 F 2 "Resistor_SMD:R_0603_1608Metric" V 6580 3775 50  0001 C CNN
 F 3 "" H 6650 3775 50  0000 C CNN
-F 4 "101-024" V 6650 3775 60  0001 C CNN "Devtank"
+F 4 "101-005" V 6650 3775 60  0001 C CNN "Devtank"
 	1    6650 3775
 	0    1    1    0
@@
 F 2 "Resistor_SMD:R_0603_1608Metric" V 4230 3550 50  0001 C CNN
 F 3 "" H 4300 3550 50  0001 C CNN
+F 4 "101-016" H 4300 3550 50  0001 C CNN "Devtank"
 	1    4300 3550
 	1    0    0    -1

Commit message: Sensi board with references visible and without stitching vias
Parts:
- C55: Dielectric (none) -> X5R; Voltage (none) -> 6.3V
- C56: Devtank 105-002 -> 105-019
Changed lines of the file:
@@
 F 3 "" H 5800 2225 50  0001 C CNN
 F 4 "105-025" H 5800 2225 50  0001 C CNN "Devtank"
+F 5 "X5R" H 5800 2225 50  0001 C CNN "Dielectric"
+F 6 "6.3V" H 5800 2225 50  0001 C CNN "Voltage"
 	1    5800 2225
 	1    0    0    -1
@@
 F 2 "Capacitor_SMD:C_0402_1005Metric" H 6263 2075 50  0001 C CNN
 F 3 "" H 6225 2225 50  0001 C CNN
-F 4 "105-002" H 6225 2225 50  0001 C CNN "Devtank"
+F 4 "105-019" H 6225 2225 50  0001 C CNN "Devtank"
 	1    6225 2225
 	1    0    0    -1

Commit message: Sensi Board Complete
Parts:
- C55: Devtank 105-025 -> 105-028
Changed lines of the file:
@@
 F 2 "Capacitor_SMD:C_0402_1005Metric" H 5838 2075 50  0001 C CNN
 F 3 "" H 5800 2225 50  0001 C CNN
-F 4 "105-025" H 5800 2225 50  0001 C CNN "Devtank"
+F 4 "105-028" H 5800 2225 50  0001 C CNN "Devtank"
 F 5 "X5R" H 5800 2225 50  0001 C CNN "Dielectric"
 F 6 "6.3V" H 5800 2225 50  0001 C CNN "Voltage"

Commit message: Rev A ordered
Parts:
- U13: footprint Package_DFN_QFN:QFN-24-1EP_4x4mm_P0.5mm_EP2.6x2.6mm_ThermalVias -> Devtank_PCB_Lib:QFN-24-1EP_4x4mm_P0.5mm_EP2.6x2.6mm_ThermalVias_0.3
Changed lines of the file:
@@
 EESchema Schematic File Version 4
 LIBS:Sensi_Board-cache
-EELAYER 30 0
+EELAYER 29 0
 EELAYER END
 $Descr A4 11693 8268
@@
 F 0 "U13" H 5125 4350 50  0000 C CNN
 F 1 "CP2102N-A01-GQFN24" H 6200 2625 50  0000 C CNN
-F 2 "Package_DFN_QFN:QFN-24-1EP_4x4mm_P0.5mm_EP2.6x2.6mm_ThermalVias" H 5975 2675 50  0001 L CNN
+F 2 "Devtank_PCB_Lib:QFN-24-1EP_4x4mm_P0.5mm_EP2.6x2.6mm_ThermalVias_0.3" H 5975 2675 50  0001 L CNN
 F 3 "http://www.silabs.com/support%20documents/technicaldocs/cp2102n-datasheet.pdf" H 5575 2425 50  0001 C CNN
 F 4 "118-007" H 5525 3475 50  0001 C CNN "Devtank"
