File: kicad_hiltop_sensi_board/USB_Debug.sch (KiCad schematic (older format))
At the start: 14 parts, among them U13 CP2102N-A01-GQFN24

Commit message: revb design updated schematics and layout
Parts:
- added C30: 100nF, Capacitor_SMD:C_0402_1005Metric, symbol device:C
- added TP20: Test_Point, TestPoint:TestPoint_THTPad_D1.0mm_Drill0.5mm, symbol Sensi_Board-rescue:Test_Point-Connector
- added U26: M74VHC1GT14DFT2G, Package_TO_SOT_SMD:SOT-353_SC-70-5, symbol Devtank:NL17SZ14
- C52: value DNF -> 100nF
- R77: value DNF -> 10k
- U13: footprint Devtank_PCB_Lib:QFN-24-1EP_4x4mm_P0.5mm_EP2.6x2.6mm_ThermalVias_0.3 -> Devtank_PCB_Lib:CP2102_QFN-24-1EP_4x4mm_P0.5mm_EP2.6x2.6mm_ThermalVias_0.3mm_drill
Connections:
- net +3V3: now also C30.2, U26.5 (VCC)
- net GND: now also C30.1, U26.3 (VSS)
- net STM_BOOT0: now also U26.4; no longer R79.1
- new net: R79.1, TP20.1, U26.2
Other:
- moved on the sheet: C52, C55, C56, R20, R76, R77, R78, R79, R80, R81, R82, R83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

Commit message: updated footprints to simplify bom
Parts:
- R77: value 10k -> 10K; Devtank (none) -> 101-010
Changed lines of the file:
@@
 P 3025 2900
 F 0 "R77" H 2900 2850 50  0000 C CNN
-F 1 "10k" H 2900 2950 50  0000 C CNN
+F 1 "10K" H 2900 2950 50  0000 C CNN
 F 2 "Resistor_SMD:R_0603_1608Metric" V 2955 2900 50  0001 C CNN
 F 3 "" H 3025 2900 50  0001 C CNN
+F 4 "101-010" H 3025 2900 50  0001 C CNN "Devtank"
 	1    3025 2900
 	-1   0    0    1
