File: kicad_hiltop_sensi_board/DigitalIO.sch (KiCad schematic (older format))
At the start: 36 parts

Commit message: Just about to aad the RTD
Parts:
- R125, R126, R127, R128, R129, R130, R131, R132, R133, R134, R135, R136, R137, R138, R139, R140, R141, R142: symbol device:R -> Sensi_Board-rescue:R-device
Changed lines of the file:
@@
 EESchema Schematic File Version 4
 LIBS:Sensi_Board-cache
-EELAYER 29 0
+EELAYER 30 0
 EELAYER END
 $Descr A3 16535 11693
 encoding utf-8
-Sheet 9 8
+Sheet 9 9
 Title "Iota Board"
 Date "2018-11-07"
@@
 	3650 3675 3800 3675
 $Comp
-L device:R R125
+L Sensi_Board-rescue:R-device R125
 U 1 1 5C6F69A0
 P 3500 3675
@@
 Max 3mA per GPIO
 $Comp
-L device:R R126
+L Sensi_Board-rescue:R-device R126
 U 1 1 5C72D67A
 P 3500 3875
@@
 $EndComp
 $Comp
-L device:R R127
+L Sensi_Board-rescue:R-device R127
 U 1 1 5C72D782
 P 3500 4075
@@
 	3125 4275 3350 4275
 $Comp
-L device:R R128
+L Sensi_Board-rescue:R-device R128
 U 1 1 5C81CFA4
 P 3500 4275
@@
 	3125 4475 3350 4475
 $Comp
-L device:R R129
+L Sensi_Board-rescue:R-device R129
 U 1 1 5C875B29
 P 3500 4475
@@
 	3125 4675 3350 4675
 $Comp
-L device:R R130
+L Sensi_Board-rescue:R-device R130
 U 1 1 5C8CEAFE
 P 3500 4675
@@
 	3700 7025 3850 7025
 $Comp
-L device:R R131
+L Sensi_Board-rescue:R-device R131
 U 1 1 5CCE0424
 P 3550 7025
@@
 	3175 7025 3400 7025
 $Comp
-L device:R R132
+L Sensi_Board-rescue:R-device R132
 U 1 1 5CCE0442
 P 3550 7225
@@
 $EndComp
 $Comp
-L device:R R133
+L Sensi_Board-rescue:R-device R133
 U 1 1 5CCE0449
 P 3550 7425
@@
 	3175 7625 3400 7625
 $Comp
-L device:R R134
+L Sensi_Board-rescue:R-device R134
 U 1 1 5CCE0460
 P 3550 7625
@@
 	3175 7825 3400 7825
 $Comp
-L device:R R135
+L Sensi_Board-rescue:R-device R135
 U 1 1 5CCE046B
 P 3550 7825
@@
 	3175 8025 3400 8025
 $Comp
-L device:R R136
+L Sensi_Board-rescue:R-device R136
 U 1 1 5CCE0476
 P 3550 8025
@@
 	9150 3675 9300 3675
 $Comp
-L device:R R137
+L Sensi_Board-rescue:R-device R137
 U 1 1 5E7ED961
 P 9000 3675
@@
 	8625 3675 8850 3675
 $Comp
-L device:R R138
+L Sensi_Board-rescue:R-device R138
 U 1 1 5E7ED97F
 P 9000 3875
@@
 $EndComp
 $Comp
-L device:R R139
+L Sensi_Board-rescue:R-device R139
 U 1 1 5E7ED986
 P 9000 4075
@@
 	8625 4275 8850 4275
 $Comp
-L device:R R140
+L Sensi_Board-rescue:R-device R140
 U 1 1 5E7ED99D
 P 9000 4275
@@
 	8625 4475 8850 4475
 $Comp
-L device:R R141
+L Sensi_Board-rescue:R-device R141
 U 1 1 5E7ED9A8
 P 9000 4475
@@
 	8625 4675 8850 4675
 $Comp
-L device:R R142
+L Sensi_Board-rescue:R-device R142
 U 1 1 5E7ED9B3
 P 9000 4675
