File: kicad_hiltop_sensi_board/DigitalIO.sch (KiCad schematic (older format))
At the start: 12 parts

Commit message: revb design updated schematics and layout
Other:
- moved on the sheet: D14A, D14B, D16A, D16B, D18A, D18B, D20A, D20B, D22A, D22B, D24A, D24B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
