File: kicad_hiltop_sensi_board/HighSideOutputs.sch (KiCad schematic (older format))
At the start: 36 parts, among them Q10 ZXMN6A07F, Q11 ZXMN6A07F, Q7 ZXMN6A07F, Q8 ZXMN6A07F, U14 BTS4140N, U15 BTS4140N, U17 BTS4140N, U18 BTS4140N

Commit message: Just about to aad the RTD
Parts:
- C57, C58, C60, C61, C63, C64, C66, C67: symbol device:C -> Sensi_Board-rescue:C-device
- L3, L4, L6, L7: symbol device:Ferrite_Bead -> Sensi_Board-rescue:Ferrite_Bead-device
- Q10, Q11, Q7, Q8: symbol device:Q_NMOS_GSD -> Sensi_Board-rescue:Q_NMOS_GSD-device
- R100, R101, R103, R104, R106, R107, R85, R86, R88, R89, R91, R92, R94, R95, R97, R98: symbol device:R -> Sensi_Board-rescue:R-device
Changed lines of the file:
@@
 EESchema Schematic File Version 4
 LIBS:Sensi_Board-cache
-EELAYER 29 0
+EELAYER 30 0
 EELAYER END
 $Descr A3 16535 11693
 encoding utf-8
-Sheet 6 8
+Sheet 6 9
 Title ""
 Date ""
@@
 $EndComp
 $Comp
-L device:Q_NMOS_GSD Q?
+L Sensi_Board-rescue:Q_NMOS_GSD-device Q?
 U 1 1 5CB48752
 P 3425 3400
@@
 $EndComp
 $Comp
-L device:R R?
+L Sensi_Board-rescue:R-device R?
 U 1 1 5CB48759
 P 2775 3400
@@
 $EndComp
 $Comp
-L device:R R?
+L Sensi_Board-rescue:R-device R?
 U 1 1 5CB48760
 P 3125 3675
@@
 	3525 3100 3525 3200
 $Comp
-L device:R R85
+L Sensi_Board-rescue:R-device R85
 U 1 1 5CB48C61
 P 2675 1750
@@
 $EndComp
 $Comp
-L device:R R91
+L Sensi_Board-rescue:R-device R91
 U 1 1 5CB48D37
 P 2950 1750
@@
 	2950 1425 2950 1600
 $Comp
-L device:Ferrite_Bead L3
+L Sensi_Board-rescue:Ferrite_Bead-device L3
 U 1 1 5CB4B291
 P 4350 2600
@@
 	3925 2600 4200 2600
 $Comp
-L device:C C60
+L Sensi_Board-rescue:C-device C60
 U 1 1 5CB4B566
 P 4775 2850
@@
 HS_CH1
 $Comp
-L device:C C57
+L Sensi_Board-rescue:C-device C57
 U 1 1 5CB4BB36
 P 2675 2450
@@
 $EndComp
 $Comp
-L device:Q_NMOS_GSD Q?
+L Sensi_Board-rescue:Q_NMOS_GSD-device Q?
 U 1 1 5CB527EB
 P 3425 6550
@@
 $EndComp
 $Comp
-L device:R R?
+L Sensi_Board-rescue:R-device R?
 U 1 1 5CB527F1
 P 2775 6550
@@
 $EndComp
 $Comp
-L device:R R?
+L Sensi_Board-rescue:R-device R?
 U 1 1 5CB527F7
 P 3125 6825
@@
 	3525 6250 3525 6350
 $Comp
-L device:R R86
+L Sensi_Board-rescue:R-device R86
 U 1 1 5CB52818
 P 2675 4900
@@
 $EndComp
 $Comp
-L device:R R92
+L Sensi_Board-rescue:R-device R92
 U 1 1 5CB5281E
 P 2950 4900
@@
 	2950 4575 2950 4750
 $Comp
-L device:Ferrite_Bead L4
+L Sensi_Board-rescue:Ferrite_Bead-device L4
 U 1 1 5CB52838
 P 4350 5750
@@
 	3925 5750 4200 5750
 $Comp
-L device:C C61
+L Sensi_Board-rescue:C-device C61
 U 1 1 5CB5283F
 P 4775 6000
@@
 HS_CH2
 $Comp
-L device:C C58
+L Sensi_Board-rescue:C-device C58
 U 1 1 5CB5284E
 P 2675 5600
@@
 $EndComp
 $Comp
-L device:Q_NMOS_GSD Q?
+L Sensi_Board-rescue:Q_NMOS_GSD-device Q?
 U 1 1 5CB58C92
 P 8475 3400
@@
 $EndComp
 $Comp
-L device:R R?
+L Sensi_Board-rescue:R-device R?
 U 1 1 5CB58C98
 P 7825 3400
@@
 $EndComp
 $Comp
-L device:R R?
+L Sensi_Board-rescue:R-device R?
 U 1 1 5CB58C9E
 P 8175 3675
@@
 	8575 3100 8575 3200
 $Comp
-L device:R R97
+L Sensi_Board-rescue:R-device R97
 U 1 1 5CB58CBF
 P 7725 1750
@@
 $EndComp
 $Comp
-L device:R R103
+L Sensi_Board-rescue:R-device R103
 U 1 1 5CB58CC5
 P 8000 1750
@@
 	8000 1425 8000 1600
 $Comp
-L device:Ferrite_Bead L6
+L Sensi_Board-rescue:Ferrite_Bead-device L6
 U 1 1 5CB58CDF
 P 9400 2600
@@
 	8975 2600 9250 2600
 $Comp
-L device:C C66
+L Sensi_Board-rescue:C-device C66
 U 1 1 5CB58CE6
 P 9825 2850
@@
 HS_CH3
 $Comp
-L device:C C63
+L Sensi_Board-rescue:C-device C63
 U 1 1 5CB58CF5
 P 7725 2450
@@
 $EndComp
 $Comp
-L device:Q_NMOS_GSD Q?
+L Sensi_Board-rescue:Q_NMOS_GSD-device Q?
 U 1 1 5CB58D11
 P 8475 6550
@@
 $EndComp
 $Comp
-L device:R R?
+L Sensi_Board-rescue:R-device R?
 U 1 1 5CB58D17
 P 7825 6550
@@
 $EndComp
 $Comp
-L device:R R?
+L Sensi_Board-rescue:R-device R?
 U 1 1 5CB58D1D
 P 8175 6825
@@
 	8575 6250 8575 6350
 $Comp
-L device:R R98
+L Sensi_Board-rescue:R-device R98
 U 1 1 5CB58D3E
 P 7725 4900
@@
 $EndComp
 $Comp
-L device:R R104
+L Sensi_Board-rescue:R-device R104
 U 1 1 5CB58D44
 P 8000 4900
@@
 	8000 4575 8000 4750
 $Comp
-L device:Ferrite_Bead L7
+L Sensi_Board-rescue:Ferrite_Bead-device L7
 U 1 1 5CB58D5E
 P 9400 5750
@@
 	8975 5750 9250 5750
 $Comp
-L device:C C67
+L Sensi_Board-rescue:C-device C67
 U 1 1 5CB58D65
 P 9825 6000
@@
 HS_CH4
 $Comp
-L device:C C64
+L Sensi_Board-rescue:C-device C64
 U 1 1 5CB58D74
 P 7725 5600
