File: kicad_hiltop_sensi_board/HighSideOutputs.sch (KiCad schematic (older format))
At the start: 36 parts, among them Q10 ZXMN6A07F, Q11 ZXMN6A07F, Q7 ZXMN6A07F, Q8 ZXMN6A07F, U14 BTS4140N, U15 BTS4140N, U17 BTS4140N, U18 BTS4140N

Commit message: revb design updated schematics and layout
Parts:
- added D1, D6, D7, D8: D_Schottky, Diode_SMD:D_SOD-123, symbol device:D_Schottky
- added R165, R166, R45, R46: 100k, Capacitor_SMD:C_0603_1608Metric, symbol device:R
Connections:
- net GND: now also D1.2 (A), D6.2 (A), D7.2 (A), D8.2 (A), R165.2, R166.2, R45.2, R46.2
- net HS_CH1: now also D1.1 (K), R45.1
- net HS_CH2: now also D6.1 (K), R46.1
- net HS_CH3: now also D7.1 (K), R165.1
- net HS_CH4: now also D8.1 (K), R166.1
Other:
- moved on the sheet: C57, C58, C60, C61, C63, C64, C66, C67, L3, L4, L6, L7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

Commit message: updated footprints to simplify bom
Parts:
- R165, R166, R45, R46: value 100k -> 100K; footprint Capacitor_SMD:C_0603_1608Metric -> Resistor_SMD:R_0603_1608Metric; Devtank (none) -> 101-015
Changed lines of the file:
@@
 P 7125 4375
 F 0 "R45" H 7195 4421 50  0000 L CNN
-F 1 "100k" H 7195 4330 50  0000 L CNN
-F 2 "Capacitor_SMD:C_0603_1608Metric" V 7055 4375 50  0001 C CNN
+F 1 "100K" H 7195 4330 50  0000 L CNN
+F 2 "Resistor_SMD:R_0603_1608Metric" V 7055 4375 50  0001 C CNN
 F 3 "" H 7125 4375 50  0001 C CNN
+F 4 "101-015" H 7125 4375 50  0001 C CNN "Devtank"
 	1    7125 4375
 	1    0    0    -1
@@
 P 12175 4375
 F 0 "R165" H 12245 4421 50  0000 L CNN
-F 1 "100k" H 12245 4330 50  0000 L CNN
-F 2 "Capacitor_SMD:C_0603_1608Metric" V 12105 4375 50  0001 C CNN
+F 1 "100K" H 12245 4330 50  0000 L CNN
+F 2 "Resistor_SMD:R_0603_1608Metric" V 12105 4375 50  0001 C CNN
 F 3 "" H 12175 4375 50  0001 C CNN
+F 4 "101-015" H 12175 4375 50  0001 C CNN "Devtank"
 	1    12175 4375
 	1    0    0    -1
@@
 P 7125 7525
 F 0 "R46" H 7195 7571 50  0000 L CNN
-F 1 "100k" H 7195 7480 50  0000 L CNN
-F 2 "Capacitor_SMD:C_0603_1608Metric" V 7055 7525 50  0001 C CNN
+F 1 "100K" H 7195 7480 50  0000 L CNN
+F 2 "Resistor_SMD:R_0603_1608Metric" V 7055 7525 50  0001 C CNN
 F 3 "" H 7125 7525 50  0001 C CNN
+F 4 "101-015" H 7125 7525 50  0001 C CNN "Devtank"
 	1    7125 7525
 	1    0    0    -1
@@
 P 12175 7525
 F 0 "R166" H 12245 7571 50  0000 L CNN
-F 1 "100k" H 12245 7480 50  0000 L CNN
-F 2 "Capacitor_SMD:C_0603_1608Metric" V 12105 7525 50  0001 C CNN
+F 1 "100K" H 12245 7480 50  0000 L CNN
+F 2 "Resistor_SMD:R_0603_1608Metric" V 12105 7525 50  0001 C CNN
 F 3 "" H 12175 7525 50  0001 C CNN
+F 4 "101-015" H 12175 7525 50  0001 C CNN "Devtank"
 	1    12175 7525
 	1    0    0    -1
