File: kicad_hiltop_sensi_board/Sensi_Board.sch (KiCad schematic (older format))
At the start: 92 parts, among them J1 Conn_02x05_Odd_Even, J2 Conn_02x03_Odd_Even, J3 Conn_03x32_DIN41612, J4 Conn_02x05_Odd_Even, J5 Conn_02x10_Odd_Even, J8 Conn_02x04_Odd_Even, U1 INA250A4, U2 LD1117S33TR_SOT223, U3 AT25DN512CSSHF-B, U6 LM75B

Commit message: Updated LBBC board and Board layout started
Parts:
- J1, J4: footprint (none) -> Connector_Molex:Molex_Pico-Clasp_501331-1007_1x10-1MP_P1.00mm_Vertical
- J2: footprint (none) -> Connector_Molex:Molex_Pico-Clasp_501331-0607_1x06-1MP_P1.00mm_Vertical
- J8: footprint (none) -> Connector_Molex:Molex_Pico-Clasp_501331-0807_1x08-1MP_P1.00mm_Vertical
Changed lines of the file:
@@
 F 0 "J8" H 4075 11992 50  0000 C CNN
 F 1 "Conn_02x04_Odd_Even" H 4075 11901 50  0000 C CNN
-F 2 "" H 4025 11675 50  0001 C CNN
+F 2 "Connector_Molex:Molex_Pico-Clasp_501331-0807_1x08-1MP_P1.00mm_Vertical" H 4025 11675 50  0001 C CNN
 F 3 "~" H 4025 11675 50  0001 C CNN
 	1    4025 11675
@@
 F 0 "J2" H 1975 11992 50  0000 C CNN
 F 1 "Conn_02x03_Odd_Even" H 1975 11901 50  0000 C CNN
-F 2 "" H 1925 11675 50  0001 C CNN
+F 2 "Connector_Molex:Molex_Pico-Clasp_501331-0607_1x06-1MP_P1.00mm_Vertical" H 1925 11675 50  0001 C CNN
 F 3 "~" H 1925 11675 50  0001 C CNN
 	1    1925 11675
@@
 F 0 "J1" H 4800 9367 50  0000 C CNN
 F 1 "Conn_02x05_Odd_Even" H 4800 9276 50  0000 C CNN
-F 2 "" H 4750 8950 50  0001 C CNN
+F 2 "Connector_Molex:Molex_Pico-Clasp_501331-1007_1x10-1MP_P1.00mm_Vertical" H 4750 8950 50  0001 C CNN
 F 3 "~" H 4750 8950 50  0001 C CNN
 	1    4750 8950
@@
 F 0 "J4" H 10150 7742 50  0000 C CNN
 F 1 "Conn_02x05_Odd_Even" H 10150 7651 50  0000 C CNN
-F 2 "" H 10100 7325 50  0001 C CNN
+F 2 "Connector_Molex:Molex_Pico-Clasp_501331-1007_1x10-1MP_P1.00mm_Vertical" H 10100 7325 50  0001 C CNN
 F 3 "~" H 10100 7325 50  0001 C CNN
 	1    10100 7325

Commit message: Started on Sensi Board Layout
Parts:
- removed J1, J4: Conn_02x05_Odd_Even, Connector_Molex:Molex_Pico-Clasp_501331-1007_1x10-1MP_P1.00mm_Vertical, symbol Connector:Conn_02x05_Odd_Even
- removed J2: Conn_02x03_Odd_Even, Connector_Molex:Molex_Pico-Clasp_501331-0607_1x06-1MP_P1.00mm_Vertical, symbol Connector:Conn_02x03_Odd_Even
- removed J5: Conn_02x10_Odd_Even, symbol Connector:Conn_02x10_Odd_Even
- removed J8: Conn_02x04_Odd_Even, Connector_Molex:Molex_Pico-Clasp_501331-0807_1x08-1MP_P1.00mm_Vertical, symbol Connector:Conn_02x04_Odd_Even
- added C24: 100nF, Capacitor_SMD:C_0603_1608Metric, symbol device:C
- added J1, J2, J4, J7, J8: Conn_01x12, Connector_Molex:Molex_Pico-Clasp_501331-1207_1x12-1MP_P1.00mm_Vertical, symbol Connector:Conn_01x12
- added J10: Conn_ARM_JTAG_SWD_10, Pin_Headers:Pin_Header_Straight_2x05_Pitch1.27mm_SMD, symbol Connector:Conn_ARM_JTAG_SWD_10
- added J5, J6: Conn_01x10, Connector_Molex:Molex_Pico-Clasp_501331-1007_1x10-1MP_P1.00mm_Vertical, symbol Connector:Conn_01x10
- added J9: Conn_01x04, Connector_Molex:Molex_Pico-Clasp_501331-0407_1x04-1MP_P1.00mm_Vertical, symbol Connector:Conn_01x04
- added R39, R40: 100K, Resistor_SMD:R_0603_1608Metric, symbol device:R
Connections:
- net labels added: SWD_IO, SWD_SCK
- wire segments 469 -> 507
- no-connect marks 65 -> 72
Other:
- note added: "EXT board Relay and GPIO\n"
- note removed: "EXT board Relay"
- moved on the sheet: R37, R38, TP3, TP4, TP5, TP55, TP56, TP57, TP58, TP6

Commit message: Updated board layout LBBC sensi board
Parts:
- removed J1, J2, J4, J7, J8: Conn_01x12, Connector_Molex:Molex_Pico-Clasp_501331-1207_1x12-1MP_P1.00mm_Vertical, symbol Connector:Conn_01x12
- removed J5, J6: Conn_01x10, Connector_Molex:Molex_Pico-Clasp_501331-1007_1x10-1MP_P1.00mm_Vertical, symbol Connector:Conn_01x10
- removed J9: Conn_01x04, Connector_Molex:Molex_Pico-Clasp_501331-0407_1x04-1MP_P1.00mm_Vertical, symbol Connector:Conn_01x04
- added J1, J2, J4, J5, J6, J7, J8: Conn_02x06_Counter_Clockwise, Devtank_PCB_Lib:Molex2x06, symbol Connector:Conn_02x06_Counter_Clockwise
- J10: footprint Pin_Headers:Pin_Header_Straight_2x05_Pitch1.27mm_SMD -> Connector_PinHeader_2.54mm:PinHeader_2x05_P2.54mm_Vertical
Connections:
- net +5V_ISO1 is gone; now on net +3V3: C23.1, C24.1, J10.1 (VCC), R30.1, R32.1, R34.1, R37.1, R38.1, R40.2, U6.8 (+Vs)
- net ADC10: now also J5.3 (Pin_3)
- net ADC11: now also J5.5 (Pin_5)
- net ADC12: now also J5.7 (Pin_7)
- net ADC9: now also J5.1 (Pin_1)
- net F1+: now also J6.1 (Pin_1)
- net F1-: now also J6.2 (Pin_2)
- net F2+: now also J6.4 (Pin_4)
- net F2-: now also J6.5 (Pin_5)
- net F3+: now also J6.11 (Pin_11)
- net F3-: now also J6.10 (Pin_10)
- net F4+: now also J6.8 (Pin_8)
- net F4-: now also J6.7 (Pin_7)
- net GND: now also J1.2 (Pin_2), J1.4 (Pin_4), J2.10 (Pin_10), J2.2 (Pin_2), J2.4 (Pin_4), J2.8 (Pin_8), J4.12 (Pin_12), J4.3 (Pin_3), J4.6 (Pin_6), J4.9 (Pin_9), J5.2 (Pin_2), J5.4 (Pin_4), J5.6 (Pin_6), J5.8 (Pin_8), J6.12 (Pin_12), J6.3 (Pin_3), J6.6 (Pin_6), J6.9 (Pin_9), J7.11 (Pin_11), J7.5 (Pin_5), J8.11 (Pin_11), J8.5 (Pin_5)
- net GPIO1: now also J1.5 (Pin_5)
- net GPIO10: now also J2.3 (Pin_3)
- net GPIO11: now also J2.5 (Pin_5)
- net GPIO12: now also J2.6 (Pin_6)
- net GPIO2: now also J1.6 (Pin_6)
- net GPIO3: now also J1.7 (Pin_7)
- net GPIO4: now also J1.8 (Pin_8)
- net GPIO5: now also J1.9 (Pin_9)
- net GPIO6: now also J1.10 (Pin_10)
- net GPIO7: now also J1.11 (Pin_11)
- net GPIO8: now also J1.12 (Pin_12)
- net GPIO9: now also J2.1 (Pin_1)
- net HS_OUT1: now also J1.1 (Pin_1)
- net HS_OUT2: now also J1.3 (Pin_3)
- net HS_OUT3: now also J2.7 (Pin_7)
- net HS_OUT4: now also J2.9 (Pin_9)
- net RTD1_F+: now also J8.1 (Pin_1)
- net RTD1_F-: now also J8.2 (Pin_2)
- net RTD1_R+: now also J8.3 (Pin_3)
- net RTD1_R-: now also J8.4 (Pin_4)
- net RTD2_F+: now also J8.7 (Pin_7)
- net RTD2_F-: now also J8.8 (Pin_8)
- net RTD2_R+: now also J8.9 (Pin_9)
- net RTD2_R-: now also J8.10 (Pin_10)
- net RTD3_F+: now also J7.1 (Pin_1)
- net RTD3_F-: now also J7.2 (Pin_2)
- net RTD3_R+: now also J7.3 (Pin_3)
- net RTD3_R-: now also J7.4 (Pin_4)
- net RTD4_F+: now also J7.7 (Pin_7)
- net RTD4_F-: now also J7.8 (Pin_8)
- net RTD4_R+: now also J7.9 (Pin_9)
- net RTD4_R-: now also J7.10 (Pin_10)
- net TH1+: now also J4.1 (Pin_1)
- net TH1-: now also J4.2 (Pin_2)
- net TH2+: now also J4.4 (Pin_4)
- net TH2-: now also J4.5 (Pin_5)
- net TH3+: now also J4.11 (Pin_11)
- net TH3-: now also J4.10 (Pin_10)
- net TH4+: now also J4.8 (Pin_8)
- net TH4-: now also J4.7 (Pin_7)
Other:
- moved on the sheet: R37, R38

Commit message: Updated sensi board layout LBBC
Connections:
- net ADC12: now also J5.12 (Pin_12); no longer J5.7 (Pin_7)
- net GND: now also J1.8 (Pin_8), J1.9 (Pin_9), J2.11 (Pin_11), J2.5 (Pin_5), J5.11 (Pin_11); no longer J1.2 (Pin_2), J1.4 (Pin_4), J2.10 (Pin_10), J2.8 (Pin_8), J5.8 (Pin_8)
- net GPIO10: now also J2.9 (Pin_9); no longer J2.3 (Pin_3)
- net GPIO11: now also J2.8 (Pin_8); no longer J2.5 (Pin_5)
- net GPIO12: now also J2.7 (Pin_7); no longer J2.6 (Pin_6)
- net GPIO3: now also J1.11 (Pin_11); no longer J1.7 (Pin_7)
- net GPIO4: now also J1.12 (Pin_12); no longer J1.8 (Pin_8)
- net GPIO5: now also J1.1 (Pin_1); no longer J1.9 (Pin_9)
- net GPIO6: now also J1.2 (Pin_2); no longer J1.10 (Pin_10)
- net GPIO7: now also J1.3 (Pin_3); no longer J1.11 (Pin_11)
- net GPIO8: now also J1.4 (Pin_4); no longer J1.12 (Pin_12)
- net GPIO9: now also J2.10 (Pin_10); no longer J2.1 (Pin_1)
- net HS_OUT1: now also J1.10 (Pin_10); no longer J1.1 (Pin_1)
- net HS_OUT2: now also J1.7 (Pin_7); no longer J1.3 (Pin_3)
- net HS_OUT3: now also J2.12 (Pin_12); no longer J2.7 (Pin_7)
- net HS_OUT4: now also J2.6 (Pin_6); no longer J2.9 (Pin_9)
Other:
- moved on the sheet: R37, R38
Changed lines of the file:
@@
 Wire Wire Line
 	12525 7775 13025 7775
+Text Label 13025 7175 2    60   ~ 0
+ADC5
+Text Label 13025 7475 2    60   ~ 0
+ADC6
+Text Label 13025 7775 2    60   ~ 0
+ADC7
 Text Label 13025 6875 2    60   ~ 0
-ADC5
-Text Label 13025 7175 2    60   ~ 0
-ADC6
-Text Label 13025 7475 2    60   ~ 0
-ADC7
-Text Label 13025 7775 2    60   ~ 0
 ADC8
 Wire Wire Line
@@
 EXT board Relay and GPIO\n
 Wire Wire Line
-	4500 11000 4150 11000
-Text Label 4150 11000 0    60   ~ 0
+	5000 11200 5350 11200
+Text Label 5350 11200 2    60   ~ 0
 GPIO9
-Text Label 4150 11200 0    60   ~ 0
+Text Label 5350 11300 2    60   ~ 0
 GPIO10
 $Comp
 L device:R R38
 U 1 1 5FD9E702
-P 3950 11200
-F 0 "R38" V 3743 11200 50  0000 C CNN
-F 1 "10K" V 3834 11200 50  0000 C CNN
-F 2 "Resistor_SMD:R_0603_1608Metric" V 3880 11200 50  0001 C CNN
-F 3 "" H 3950 11200 50  0001 C CNN
-	1    3950 11200
-	0    -1   1    0
+P 5550 11300
+F 0 "R38" V 5343 11300 50  0000 C CNN
+F 1 "10K" V 5434 11300 50  0000 C CNN
+F 2 "Resistor_SMD:R_0603_1608Metric" V 5480 11300 50  0001 C CNN
+F 3 "" H 5550 11300 50  0001 C CNN
+	1    5550 11300
+	0    1    1    0
 $EndComp
 $Comp
 L device:R R37
 U 1 1 5FD9EAEE
-P 4150 10775
-F 0 "R37" H 4220 10821 50  0000 L CNN
-F 1 "10K" H 4220 10730 50  0000 L CNN
-F 2 "Resistor_SMD:R_0603_1608Metric" V 4080 10775 50  0001 C CNN
-F 3 "" H 4150 10775 50  0001 C CNN
-	1    4150 10775
-	-1   0    0    -1
-$EndComp
-Wire Wire Line
-	3800 11200 3775 11200
-Wire Wire Line
-	3775 11200 3775 11125
-Wire Wire Line
-	4500 11200 4100 11200
-Wire Wire Line
-	4150 11000 4150 10925
-Wire Wire Line
-	4150 10625 4150 10550
+P 5350 10650
+F 0 "R37" H 5420 10696 50  0000 L CNN
+F 1 "10K" H 5420 10605 50  0000 L CNN
+F 2 "Resistor_SMD:R_0603_1608Metric" V 5280 10650 50  0001 C CNN
+F 3 "" H 5350 10650 50  0001 C CNN
+	1    5350 10650
+	1    0    0    -1
+$EndComp
+Wire Wire Line
+	5700 11300 5725 11300
+Wire Wire Line
+	5725 11300 5725 11225
+Wire Wire Line
+	5000 11300 5400 11300
+Wire Wire Line
+	5350 10500 5350 10425
 Text Notes 4500 11750 0    60   ~ 0
 Shot Bolt
@@
 Wire Wire Line
 	5225 8750 5700 8750
-Text Label 1350 11125 0    60   ~ 0
+Text Label 2575 11325 2    60   ~ 0
 HS_OUT1
 Wire Wire Line
 	1350 11125 1750 11125
-Text Label 1350 11325 0    60   ~ 0
+Text Label 2650 11625 2    60   ~ 0
 HS_OUT2
 Wire Wire Line
-	1750 11325 1350 11325
+	2250 11625 2650 11625
 Wire Wire Line
 	1750 11525 1425 11525
@@
 	1750 11625 1425 11625
 Wire Wire Line
-	2250 11625 2575 11625
-Wire Wire Line
-	2250 11525 2575 11525
-Wire Wire Line
-	2250 11425 2575 11425
+	2250 11125 2575 11125
 Wire Wire Line
 	2250 11325 2575 11325
 Wire Wire Line
-	2250 11225 2575 11225
-Wire Wire Line
-	2250 11125 2575 11125
+	2250 11425 2325 11425
+Wire Wire Line
+	1750 11425 1425 11425
+Wire Wire Line
+	1750 11325 1425 11325
 Text Label 1425 11525 0    60   ~ 0
 GPIO1
-Text Label 2575 11625 2    60   ~ 0
+Text Label 2575 11225 2    60   ~ 0
 GPIO3
-Text Label 2575 11525 2    60   ~ 0
+Text Label 2575 11125 2    60   ~ 0
 GPIO4
-Text Label 2575 11425 2    60   ~ 0
+Text Label 1350 11125 0    60   ~ 0
 GPIO5
-Text Label 2575 11325 2    60   ~ 0
+Text Label 1350 11225 0    60   ~ 0
 GPIO6
-Text Label 2575 11225 2    60   ~ 0
+Text Label 1425 11325 0    60   ~ 0
 GPIO7
-Text Label 2575 11125 2    60   ~ 0
+Text Label 1425 11425 0    60   ~ 0
 GPIO8
 Text Label 1425 11625 0    60   ~ 0
 GPIO2
 Wire Wire Line
-	5000 11300 5600 11300
-Text Label 5600 11300 2    60   ~ 0
+	4500 11500 3900 11500
+Text Label 3900 11500 0    60   ~ 0
 HS_OUT4
 Wire Wire Line
-	5000 11500 5425 11500
-Text Label 5425 11500 2    60   ~ 0
+	5000 11000 5425 11000
+Text Label 5425 11000 2    60   ~ 0
 HS_OUT3
 $Comp
@@
 	-1   0    0    -1
 $EndComp
-Text Label 4075 11400 0    60   ~ 0
+Text Label 5425 11400 2    60   ~ 0
 GPIO11
 Wire Wire Line
-	4500 11400 4075 11400
-Wire Wire Line
-	4500 11500 4075 11500
-Text Label 4075 11500 0    60   ~ 0
+	5000 11400 5425 11400
+Wire Wire Line
+	5000 11500 5425 11500
+Text Label 5425 11500 2    60   ~ 0
 GPIO12
 Wire Wire Line
@@
 L power:+3V3 #PWR0113
 U 1 1 5E269C11
-P 4150 10550
-F 0 "#PWR0113" H 4150 10400 50  0001 C CNN
-F 1 "+3V3" H 4165 10723 50  0000 C CNN
-F 2 "" H 4150 10550 50  0001 C CNN
-F 3 "" H 4150 10550 50  0001 C CNN
-	1    4150 10550
-	-1   0    0    -1
+P 5350 10425
+F 0 "#PWR0113" H 5350 10275 50  0001 C CNN
+F 1 "+3V3" H 5365 10598 50  0000 C CNN
+F 2 "" H 5350 10425 50  0001 C CNN
+F 3 "" H 5350 10425 50  0001 C CNN
+	1    5350 10425
+	1    0    0    -1
 $EndComp
 $Comp
 L power:+3V3 #PWR0118
 U 1 1 5E41062F
-P 3775 11125
-F 0 "#PWR0118" H 3775 10975 50  0001 C CNN
-F 1 "+3V3" H 3790 11298 50  0000 C CNN
-F 2 "" H 3775 11125 50  0001 C CNN
-F 3 "" H 3775 11125 50  0001 C CNN
-	1    3775 11125
-	-1   0    0    -1
+P 5725 11225
+F 0 "#PWR0118" H 5725 11075 50  0001 C CNN
+F 1 "+3V3" H 5740 11398 50  0000 C CNN
+F 2 "" H 5725 11225 50  0001 C CNN
+F 3 "" H 5725 11225 50  0001 C CNN
+	1    5725 11225
+	1    0    0    -1
 $EndComp
 $Comp
@@
 L power:GND #PWR0257
 U 1 1 5F845C63
-P 5125 11625
-F 0 "#PWR0257" H 5125 11375 50  0001 C CNN
-F 1 "GND" H 5130 11452 50  0000 C CNN
-F 2 "" H 5125 11625 50  0001 C CNN
-F 3 "" H 5125 11625 50  0001 C CNN
-	1    5125 11625
+P 5200 11600
+F 0 "#PWR0257" H 5200 11350 50  0001 C CNN
+F 1 "GND" H 5205 11427 50  0000 C CNN
+F 2 "" H 5200 11600 50  0001 C CNN
+F 3 "" H 5200 11600 50  0001 C CNN
+	1    5200 11600
 	-1   0    0    -1
 $EndComp
-Wire Wire Line
-	5000 11200 5125 11200
-Wire Wire Line
-	5000 11400 5125 11400
 Wire Wire Line
 	12550 9975 12125 9975
@@
 ADC11
 Wire Wire Line
-	7450 14725 7875 14725
-$Comp
-L power:GND #PWR0254
-U 1 1 5E2F6AA1
-P 8025 14625
-F 0 "#PWR0254" H 8025 14375 50  0001 C CNN
-F 1 "GND" H 8030 14452 50  0000 C CNN
-F 2 "" H 8025 14625 50  0001 C CNN
-F 3 "" H 8025 14625 50  0001 C CNN
-	1    8025 14625
-	1    0    0    -1
-$EndComp
-Wire Wire Line
-	7450 14625 8025 14625
-Text Label 7875 14725 2    60   ~ 0
+	7450 14225 7875 14225
+Text Label 7875 14225 2    60   ~ 0
 ADC12
 NoConn ~ 7450 14525
 NoConn ~ 7450 14425
-NoConn ~ 7450 14325
-NoConn ~ 7450 14225
 $Comp
 L Connector:Conn_02x06_Counter_Clockwise J6
@@
 	-1   0    0    -1
 $EndComp
-NoConn ~ 5000 11000
-NoConn ~ 5000 11100
 Wire Wire Line
 	10300 7100 10350 7100
@@
 $EndComp
 Wire Wire Line
-	5125 11200 5125 11400
-Connection ~ 5125 11400
-Wire Wire Line
-	5125 11400 5125 11625
-Wire Wire Line
-	4500 11300 4325 11300
-Wire Wire Line
-	4325 11300 4325 11650
-Wire Wire Line
 	4500 11100 4325 11100
-Wire Wire Line
-	4325 11100 4325 11300
-Connection ~ 4325 11300
-$Comp
-L power:GND #PWR0203
-U 1 1 5FC4F4B6
-P 1675 11725
-F 0 "#PWR0203" H 1675 11475 50  0001 C CNN
-F 1 "GND" H 1680 11552 50  0000 C CNN
-F 2 "" H 1675 11725 50  0001 C CNN
-F 3 "" H 1675 11725 50  0001 C CNN
-	1    1675 11725
-	1    0    0    -1
-$EndComp
-Wire Wire Line
-	1750 11225 1675 11225
-Wire Wire Line
-	1675 11225 1675 11425
-Wire Wire Line
-	1750 11425 1675 11425
-Connection ~ 1675 11425
-Wire Wire Line
-	1675 11425 1675 11725
 Wire Wire Line
 	6950 14325 6825 14325
@@
 	1    0    0    -1
 $EndComp
+Wire Wire Line
+	1750 11225 1350 11225
+Wire Wire Line
+	2250 11525 2325 11525
+Wire Wire Line
+	2250 11225 2575 11225
+Wire Wire Line
+	2325 11525 2325 11425
+$Comp
+L power:GND #PWR0203
+U 1 1 5E41A061
+P 2325 11725
+F 0 "#PWR0203" H 2325 11475 50  0001 C CNN
+F 1 "GND" H 2330 11552 50  0000 C CNN
+F 2 "" H 2325 11725 50  0001 C CNN
+F 3 "" H 2325 11725 50  0001 C CNN
+	1    2325 11725
+	1    0    0    -1
+$EndComp
+Wire Wire Line
+	2325 11525 2325 11725
+Connection ~ 2325 11525
+Wire Wire Line
+	4325 11100 4325 11300
+Wire Wire Line
+	4500 11400 4325 11400
+Connection ~ 4325 11400
+Wire Wire Line
+	4325 11400 4325 11650
+Wire Wire Line
+	4500 11300 4325 11300
+Connection ~ 4325 11300
+Wire Wire Line
+	4325 11300 4325 11400
+Wire Wire Line
+	5000 11100 5200 11100
+Wire Wire Line
+	5200 11100 5200 11600
+Wire Wire Line
+	5350 10800 5350 11200
+NoConn ~ 4500 11000
+NoConn ~ 4500 11200
+$Comp
+L power:GND #PWR0254
+U 1 1 5DABC198
+P 7625 14325
+F 0 "#PWR0254" H 7625 14075 50  0001 C CNN
+F 1 "GND" H 7630 14152 50  0000 C CNN
+F 2 "" H 7625 14325 50  0001 C CNN
+F 3 "" H 7625 14325 50  0001 C CNN
+	1    7625 14325
+	1    0    0    -1
+$EndComp
+Wire Wire Line
+	7450 14325 7625 14325
+NoConn ~ 7450 14625
+NoConn ~ 7450 14725
 $EndSCHEMATC

Commit message: Sensi board updated pin map
Parts:
- C12, C23, C24, C9: footprint Capacitor_SMD:C_0603_1608Metric -> Capacitor_SMD:C_0402_1005Metric
Connections:
- no-connect marks 72 -> 74
Changed lines of the file:
@@
 F 0 "C9" V 18323 10050 50  0000 C CNN
 F 1 "100nF" V 18414 10050 50  0000 C CNN
-F 2 "Capacitor_SMD:C_0603_1608Metric" H 18613 9900 50  0001 C CNN
+F 2 "Capacitor_SMD:C_0402_1005Metric" H 18613 9900 50  0001 C CNN
 F 3 "" H 18575 10050 50  0001 C CNN
 F 4 "105-002" H -350 1050 50  0001 C CNN "Devtank"
@@
 F 0 "C12" V 21623 3125 50  0000 C CNN
 F 1 "100nF" V 21714 3125 50  0000 C CNN
-F 2 "Capacitor_SMD:C_0603_1608Metric" H 21913 2975 50  0001 C CNN
+F 2 "Capacitor_SMD:C_0402_1005Metric" H 21913 2975 50  0001 C CNN
 F 3 "" H 21875 3125 50  0001 C CNN
 F 4 "105-002" H 0   0   50  0001 C CNN "Devtank"
@@
 Wire Wire Line
 	12525 7775 13025 7775
-Text Label 13025 7175 2    60   ~ 0
+Text Label 13025 7775 2    60   ~ 0
 ADC5
 Text Label 13025 7475 2    60   ~ 0
 ADC6
-Text Label 13025 7775 2    60   ~ 0
+Text Label 13025 7175 2    60   ~ 0
 ADC7
 Text Label 13025 6875 2    60   ~ 0
@@
 Text Label 8350 9450 2    60   ~ 0
 ADC4
-Text Label 8350 9150 2    60   ~ 0
-ADC3
 Text Label 8350 8850 2    60   ~ 0
-ADC2
+ADC3
 Text Label 8350 8550 2    60   ~ 0
+ADC2
+Text Label 8350 9150 2    60   ~ 0
 ADC1
 Wire Wire Line
@@
 Text Label 8675 14750 0    60   ~ 0
 5V_ADC12
-Text Label 11100 14300 2    60   ~ 0
-ADC9
-Text Label 11100 14450 2    60   ~ 0
-ADC10
-Text Label 11100 14600 2    60   ~ 0
-ADC11
 Text Label 11100 14750 2    60   ~ 0
 ADC12
@@
 F 0 "C23" V 8952 10975 50  0000 C CNN
 F 1 "100nF" V 8861 10975 50  0000 C CNN
-F 2 "Capacitor_SMD:C_0603_1608Metric" H 8738 10825 50  0001 C CNN
+F 2 "Capacitor_SMD:C_0402_1005Metric" H 8738 10825 50  0001 C CNN
 F 3 "" H 8700 10975 50  0001 C CNN
 	1    8700 10975
@@
 F 0 "C24" H 1065 8496 50  0000 L CNN
 F 1 "100nF" H 1065 8405 50  0000 L CNN
-F 2 "Capacitor_SMD:C_0603_1608Metric" H 988 8300 50  0001 C CNN
+F 2 "Capacitor_SMD:C_0402_1005Metric" H 988 8300 50  0001 C CNN
 F 3 "" H 950 8450 50  0001 C CNN
 	1    950  8450
@@
 NoConn ~ 7450 14625
 NoConn ~ 7450 14725
+Text Label 11100 14600 2    60   ~ 0
+ADC11
+Text Label 11100 14450 2    60   ~ 0
+ADC10
+Text Label 11100 14300 2    60   ~ 0
+ADC9
+Wire Wire Line
+	3225 6775 2525 6775
+Wire Wire Line
+	3225 6900 2525 6900
+NoConn ~ 2525 6775
+NoConn ~ 2525 6900
 $EndSCHEMATC
