File: kicad_hiltop_sensi_board/Sensi_Board.sch (KiCad schematic (older format))
At the start: 151 parts, among them J1 Conn_02x06_Top_Bottom, J10 Conn_02x05_Counter_Clockwise, J2 Conn_02x06_Top_Bottom, J3 Conn_03x32_DIN41612, J4 Conn_02x06_Top_Bottom, J5 Conn_02x06_Top_Bottom, J6 Conn_02x10_Counter_Clockwise, J7 Conn_02x06_Top_Bottom, J8 Conn_02x06_Top_Bottom, J9 Conn_02x06_Top_Bottom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

Commit message: revb design updated schematics and layout
Parts:
- removed C30: 100nF, Capacitor_SMD:C_0402_1005Metric, symbol device:C
- removed J10: Conn_02x05_Counter_Clockwise, Connector_PinHeader_2.54mm:PinHeader_2x05_P2.54mm_Vertical, symbol Connector:Conn_02x05_Counter_Clockwise
- removed J6: Conn_02x10_Counter_Clockwise, Devtank_PCB_Lib:Molex_Milligrid_2x10, symbol Connector:Conn_02x10_Counter_Clockwise
- removed J7, J8, J9: Conn_02x06_Top_Bottom, Devtank_PCB_Lib:Molex2x06, symbol Connector:Conn_02x06_Top_Bottom
- removed R39, R40: 100K, Resistor_SMD:R_0603_1608Metric, symbol device:R
- removed R45: DNF, Resistor_SMD:R_0805_2012Metric, symbol device:R
- removed R46: 0R, Resistor_SMD:R_0805_2012Metric, symbol device:R
- added J11: Conn_02x10_Counter_Clockwise, Devtank_PCB_Lib:Molex_Milligrid_2x10, symbol Connector:Conn_02x10_Counter_Clockwise
- added J6: Conn_02x06_Top_Bottom, Devtank_PCB_Lib:Molex2x06, symbol Connector:Conn_02x06_Top_Bottom
- added J7, J8: Conn_02x07_Top_Bottom, Devtank_PCB_Lib:87831-1420_Molex_Milligrid, symbol Connector:Conn_02x07_Top_Bottom
- added R167, R168, R169: DNF, Capacitor_SMD:C_0603_1608Metric, symbol device:R
- added R170: 10K, Resistor_SMD:R_0603_1608Metric, symbol device:R
- added R171: 1k5, Resistor_SMD:R_0603_1608Metric, symbol device:R
- C24, C26, C27, C28, C29: Devtank 105-019 -> (none)
- JP2, JP3, JP4, JP5: Devtank 714-005 -> (none)
- R38: value 10K -> DNF; footprint Resistor_SMD:R_0603_1608Metric -> Capacitor_SMD:C_0603_1608Metric; Devtank 101-010 -> (none)
- R41: value DNF -> R; footprint Resistor_SMD:R_0805_2012Metric -> Capacitor_SMD:C_0805_2012Metric
- R44: value 0R -> R; footprint Resistor_SMD:R_0805_2012Metric -> Capacitor_SMD:C_0805_2012Metric; Devtank 101-006 -> (none)
Connections:
- net labels added: F_Vs, STM_BOOT0_OUT
- net labels removed: STM_BOOT0
- wire segments 614 -> 586
- no-connect marks 72 -> 64
Other:
- note added: "3.3V Regulator\n"
- note added: "4 Channels of 4-20mA \n"
- note added: "4 Channels of Analogue Inputs (0-5V)\n"
- note added: "4 Channels of RTD\n"
- note added: "4 Channels of Thermocouple\n"
- note added: "4 High Side Switches\n"
- note added: "6x GPIO's"
- note added: "96Way Backplane Connector"
- note added: "Misc Connectors"
- note added: "NOTE: Fit 1k5 for 303/302 model. DNF for 072 model"
- note added: "Onboard EEPROM\n"
- note added: "Onboard temperature sensor"
- note added: "Optional 3v3 from either backplane or onboard regulator"
- note added: "Relay + PSU O/P Connector\n"
- note added: "Relay Output"
- note added: "STM Microcontroller\n"
- note added: "USB Debug"
- note added: "USB Hub Controller"
- note removed: "4-20mA"
- note removed: "4off High side switches (12/24V)\n4off RTD's\n4off thermocouple\n4off 4-20mA\n4off 0-5V analogue \n6off digital inputs\n6off digital outputs\n\n"
- note removed: "Analogue Inputs\n"
- note removed: "JTAG Header\n"
- note removed: "Relay + PSU O/P\n"
- moved on the sheet: C10, C11, C12, C13, C23, C9, D32, F1, J1, J2, J3A, J3B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

Commit message: revB ready for review
Parts:
- R41: value R -> DNF
- R44: value R -> 0R
Connections:
- net SB1 renamed GPIO5
- net SB2 renamed GPIO6
Changed lines of the file:
@@
 Wire Wire Line
 	2725 5900 1675 5900
-Text Label 1675 5900 0    60   ~ 0
-SB2
 Text Label 1675 6025 0    60   ~ 0
 GPIO1
@@
 Wire Wire Line
 	4100 15475 5225 15475
-Text Label 5000 15325 2    60   ~ 0
-SB1
-Text Label 5000 15475 2    60   ~ 0
-SB2
 Text Label 1125 14725 0    60   ~ 0
 GPIO1_EXT
@@
 Text Label 1675 4900 0    60   ~ 0
 RTD1_CS
-Text Label 1675 5775 0    60   ~ 0
-SB1
 Text Label 1675 5400 0    60   ~ 0
 RTD3_CS
@@
 F41 "RTD2_INT" B L 2725 5025 60
 F42 "RTD3_CS" B L 2725 5400 60
-F43 "SB2" B L 2725 5900 60
-F44 "SB1" B L 2725 5775 60
-F45 "GPIO1" B L 2725 6025 60
-F46 "GPIO2" B L 2725 6150 60
-F47 "GPIO3" B L 2725 6250 60
-F48 "GPIO4" B L 2725 6360 60
+F43 "GPIO1" B L 2725 6025 60
+F44 "GPIO2" B L 2725 6150 60
+F45 "GPIO3" B L 2725 6250 60
+F46 "GPIO4" B L 2725 6360 60
+F47 "GPIO6" B L 2725 5900 60
+F48 "GPIO5" B L 2725 5775 60
 $EndSheet
 Wire Wire Line
@@
 P 7975 8525
 F 0 "R41" H 7905 8479 50  0000 R CNN
-F 1 "R" H 7905 8570 50  0000 R CNN
+F 1 "DNF" H 7905 8570 50  0000 R CNN
 F 2 "Capacitor_SMD:C_0805_2012Metric" V 7905 8525 50  0001 C CNN
 F 3 "" H 7975 8525 50  0001 C CNN
@@
 P 8300 8525
 F 0 "R44" H 8230 8479 50  0000 R CNN
-F 1 "R" H 8230 8570 50  0000 R CNN
+F 1 "0R" H 8230 8570 50  0000 R CNN
 F 2 "Capacitor_SMD:C_0805_2012Metric" V 8230 8525 50  0001 C CNN
 F 3 "" H 8300 8525 50  0001 C CNN
@@
 	1    0    0    -1
 $EndComp
-Wire Wire Line
-	8025 9625 7675 9625
-Text Label 7675 9625 0    60   ~ 0
-F1_OUT
-Wire Wire Line
-	8025 9225 7675 9225
-Text Label 7675 9225 0    60   ~ 0
-F2_OUT
 $Comp
 L power:GND #PWR0115
@@
 Text Label 8875 9325 2    60   ~ 0
 F4+
-Text Label 8875 9425 2    60   ~ 0
-F4_OUT
-Wire Wire Line
-	8525 9425 8875 9425
-Text Label 8875 9825 2    60   ~ 0
-F3_OUT
-Wire Wire Line
-	8525 9825 8875 9825
 $Comp
 L device:R R38
@@
 	-1   0    0    -1
 $EndComp
+Text Label 7675 9225 0    60   ~ 0
+F2_OUT
+Wire Wire Line
+	8025 9225 7675 9225
+Text Label 7675 9625 0    60   ~ 0
+F1_OUT
+Wire Wire Line
+	8025 9625 7675 9625
+Wire Wire Line
+	8525 9825 8875 9825
+Text Label 8875 9825 2    60   ~ 0
+F3_OUT
+Wire Wire Line
+	8525 9425 8875 9425
+Text Label 8875 9425 2    60   ~ 0
+F4_OUT
+Text Label 5000 15325 2    60   ~ 0
+GPIO5
+Text Label 5000 15475 2    60   ~ 0
+GPIO6
+Text Label 1675 5775 0    60   ~ 0
+GPIO5
+Text Label 1675 5900 0    60   ~ 0
+GPIO6
 $EndSCHEMATC

Commit message: updated footprints to simplify bom
Parts:
- R167, R168, R169, R38: footprint Capacitor_SMD:C_0603_1608Metric -> Resistor_SMD:R_0603_1608Metric
- R41, R44: footprint Capacitor_SMD:C_0805_2012Metric -> Resistor_SMD:R_0805_2012Metric
Changed lines of the file:
@@
 F 0 "R41" H 7905 8479 50  0000 R CNN
 F 1 "DNF" H 7905 8570 50  0000 R CNN
-F 2 "Capacitor_SMD:C_0805_2012Metric" V 7905 8525 50  0001 C CNN
+F 2 "Resistor_SMD:R_0805_2012Metric" V 7905 8525 50  0001 C CNN
 F 3 "" H 7975 8525 50  0001 C CNN
 	1    7975 8525
@@
 F 0 "R44" H 8230 8479 50  0000 R CNN
 F 1 "0R" H 8230 8570 50  0000 R CNN
-F 2 "Capacitor_SMD:C_0805_2012Metric" V 8230 8525 50  0001 C CNN
+F 2 "Resistor_SMD:R_0805_2012Metric" V 8230 8525 50  0001 C CNN
 F 3 "" H 8300 8525 50  0001 C CNN
 	1    8300 8525
@@
 F 0 "R38" H 19450 9000 50  0000 L CNN
 F 1 "DNF" H 19450 8900 50  0000 L CNN
-F 2 "Capacitor_SMD:C_0603_1608Metric" V 19330 8950 50  0001 C CNN
+F 2 "Resistor_SMD:R_0603_1608Metric" V 19330 8950 50  0001 C CNN
 F 3 "" H 19400 8950 50  0001 C CNN
 	1    19400 8950
@@
 F 0 "R167" H 19750 9000 50  0000 L CNN
 F 1 "DNF" H 19750 8900 50  0000 L CNN
-F 2 "Capacitor_SMD:C_0603_1608Metric" V 19630 8950 50  0001 C CNN
+F 2 "Resistor_SMD:R_0603_1608Metric" V 19630 8950 50  0001 C CNN
 F 3 "" H 19700 8950 50  0001 C CNN
 	1    19700 8950
@@
 F 0 "R168" H 20050 9000 50  0000 L CNN
 F 1 "DNF" H 20050 8900 50  0000 L CNN
-F 2 "Capacitor_SMD:C_0603_1608Metric" V 19930 8950 50  0001 C CNN
+F 2 "Resistor_SMD:R_0603_1608Metric" V 19930 8950 50  0001 C CNN
 F 3 "" H 20000 8950 50  0001 C CNN
 	1    20000 8950
@@
 F 0 "R169" H 20350 9000 50  0000 L CNN
 F 1 "DNF" H 20350 8900 50  0000 L CNN
-F 2 "Capacitor_SMD:C_0603_1608Metric" V 20230 8950 50  0001 C CNN
+F 2 "Resistor_SMD:R_0603_1608Metric" V 20230 8950 50  0001 C CNN
 F 3 "" H 20300 8950 50  0001 C CNN
 	1    20300 8950
