File: kicad_hiltop_sensi_board/RTDinputs.sch (KiCad schematic (older format))
At the start: 28 parts, among them SW2 SW_DIP_x04, SW3 SW_DIP_x04, SW4 SW_DIP_x04, SW5 SW_DIP_x04, U10 MAX31865, U11 MAX31865, U8 MAX31865, U9 MAX31865

Commit message: Updated LBBC board and Board layout started
Parts:
- SW2, SW3, SW4, SW5: footprint (none) -> Button_Switch_SMD:SW_DIP_SPSTx04_Slide_6.7x11.72mm_W6.73mm_P2.54mm_LowProfile_JPin
- U10, U11, U8, U9: footprint (none) -> Package_DFN_QFN:TQFN-20-1EP_5x5mm_P0.65mm_EP3.1x3.1mm
Changed lines of the file:
@@
 F 0 "U10" H 2850 3650 60  0000 C CNN
 F 1 "MAX31865" H 3000 3550 60  0000 C CNN
-F 2 "" H 3150 2800 60  0001 C CNN
+F 2 "Package_DFN_QFN:TQFN-20-1EP_5x5mm_P0.65mm_EP3.1x3.1mm" H 3150 2800 60  0001 C CNN
 F 3 "" H 3150 2800 60  0001 C CNN
 	1    3400 2750
@@
 F 0 "SW2" H 3425 5117 50  0000 C CNN
 F 1 "SW_DIP_x04" H 3425 5026 50  0000 C CNN
-F 2 "" H 3425 4650 50  0001 C CNN
+F 2 "Button_Switch_SMD:SW_DIP_SPSTx04_Slide_6.7x11.72mm_W6.73mm_P2.54mm_LowProfile_JPin" H 3425 4650 50  0001 C CNN
 F 3 "" H 3425 4650 50  0001 C CNN
 	1    3425 4650
@@
 F 0 "U11" H 6675 3625 60  0000 C CNN
 F 1 "MAX31865" H 6825 3525 60  0000 C CNN
-F 2 "" H 6975 2775 60  0001 C CNN
+F 2 "Package_DFN_QFN:TQFN-20-1EP_5x5mm_P0.65mm_EP3.1x3.1mm" H 6975 2775 60  0001 C CNN
 F 3 "" H 6975 2775 60  0001 C CNN
 	1    7225 2725
@@
 F 0 "SW5" H 7250 5092 50  0000 C CNN
 F 1 "SW_DIP_x04" H 7250 5001 50  0000 C CNN
-F 2 "" H 7250 4625 50  0001 C CNN
+F 2 "Button_Switch_SMD:SW_DIP_SPSTx04_Slide_6.7x11.72mm_W6.73mm_P2.54mm_LowProfile_JPin" H 7250 4625 50  0001 C CNN
 F 3 "" H 7250 4625 50  0001 C CNN
 	1    7250 4625
@@
 F 0 "U8" H 2850 8375 60  0000 C CNN
 F 1 "MAX31865" H 3000 8275 60  0000 C CNN
-F 2 "" H 3150 7525 60  0001 C CNN
+F 2 "Package_DFN_QFN:TQFN-20-1EP_5x5mm_P0.65mm_EP3.1x3.1mm" H 3150 7525 60  0001 C CNN
 F 3 "" H 3150 7525 60  0001 C CNN
 	1    3400 7475
@@
 F 0 "SW3" H 3425 9842 50  0000 C CNN
 F 1 "SW_DIP_x04" H 3425 9751 50  0000 C CNN
-F 2 "" H 3425 9375 50  0001 C CNN
+F 2 "Button_Switch_SMD:SW_DIP_SPSTx04_Slide_6.7x11.72mm_W6.73mm_P2.54mm_LowProfile_JPin" H 3425 9375 50  0001 C CNN
 F 3 "" H 3425 9375 50  0001 C CNN
 	1    3425 9375
@@
 F 0 "U9" H 6650 8275 60  0000 C CNN
 F 1 "MAX31865" H 6800 8175 60  0000 C CNN
-F 2 "" H 6950 7425 60  0001 C CNN
+F 2 "Package_DFN_QFN:TQFN-20-1EP_5x5mm_P0.65mm_EP3.1x3.1mm" H 6950 7425 60  0001 C CNN
 F 3 "" H 6950 7425 60  0001 C CNN
 	1    7200 7375
@@
 F 0 "SW4" H 7225 9742 50  0000 C CNN
 F 1 "SW_DIP_x04" H 7225 9651 50  0000 C CNN
-F 2 "" H 7225 9275 50  0001 C CNN
+F 2 "Button_Switch_SMD:SW_DIP_SPSTx04_Slide_6.7x11.72mm_W6.73mm_P2.54mm_LowProfile_JPin" H 7225 9275 50  0001 C CNN
 F 3 "" H 7225 9275 50  0001 C CNN
 	1    7225 9275

Commit message: Updated board layout LBBC sensi board
Parts:
- SW2, SW3, SW4, SW5: footprint Button_Switch_SMD:SW_DIP_SPSTx04_Slide_6.7x11.72mm_W6.73mm_P2.54mm_LowProfile_JPin -> Button_Switch_SMD:SW_DIP_SPSTx04_Slide_Copal_CHS-04B_W7.62mm_P1.27mm
Changed lines of the file:
@@
 F 0 "SW2" H 3425 5117 50  0000 C CNN
 F 1 "SW_DIP_x04" H 3425 5026 50  0000 C CNN
-F 2 "Button_Switch_SMD:SW_DIP_SPSTx04_Slide_6.7x11.72mm_W6.73mm_P2.54mm_LowProfile_JPin" H 3425 4650 50  0001 C CNN
+F 2 "Button_Switch_SMD:SW_DIP_SPSTx04_Slide_Copal_CHS-04B_W7.62mm_P1.27mm" H 3425 4650 50  0001 C CNN
 F 3 "" H 3425 4650 50  0001 C CNN
 	1    3425 4650
@@
 F 0 "SW5" H 7250 5092 50  0000 C CNN
 F 1 "SW_DIP_x04" H 7250 5001 50  0000 C CNN
-F 2 "Button_Switch_SMD:SW_DIP_SPSTx04_Slide_6.7x11.72mm_W6.73mm_P2.54mm_LowProfile_JPin" H 7250 4625 50  0001 C CNN
+F 2 "Button_Switch_SMD:SW_DIP_SPSTx04_Slide_Copal_CHS-04B_W7.62mm_P1.27mm" H 7250 4625 50  0001 C CNN
 F 3 "" H 7250 4625 50  0001 C CNN
 	1    7250 4625
@@
 F 0 "SW3" H 3425 9842 50  0000 C CNN
 F 1 "SW_DIP_x04" H 3425 9751 50  0000 C CNN
-F 2 "Button_Switch_SMD:SW_DIP_SPSTx04_Slide_6.7x11.72mm_W6.73mm_P2.54mm_LowProfile_JPin" H 3425 9375 50  0001 C CNN
+F 2 "Button_Switch_SMD:SW_DIP_SPSTx04_Slide_Copal_CHS-04B_W7.62mm_P1.27mm" H 3425 9375 50  0001 C CNN
 F 3 "" H 3425 9375 50  0001 C CNN
 	1    3425 9375
@@
 F 0 "SW4" H 7225 9742 50  0000 C CNN
 F 1 "SW_DIP_x04" H 7225 9651 50  0000 C CNN
-F 2 "Button_Switch_SMD:SW_DIP_SPSTx04_Slide_6.7x11.72mm_W6.73mm_P2.54mm_LowProfile_JPin" H 7225 9275 50  0001 C CNN
+F 2 "Button_Switch_SMD:SW_DIP_SPSTx04_Slide_Copal_CHS-04B_W7.62mm_P1.27mm" H 7225 9275 50  0001 C CNN
 F 3 "" H 7225 9275 50  0001 C CNN
 	1    7225 9275

Commit message: Updated sensi board layout LBBC
Parts:
- C1: footprint Capacitor_SMD:C_0603_1608Metric -> Crystal:Crystal_SMD_TXC_7A-2Pin_5x3.2mm
Changed lines of the file:
@@
 F 0 "C1" V 3150 8825 50  0000 C CNN
 F 1 "100n" V 3239 8775 50  0000 C CNN
-F 2 "Capacitor_SMD:C_0603_1608Metric" H 3438 8625 50  0001 C CNN
+F 2 "Crystal:Crystal_SMD_TXC_7A-2Pin_5x3.2mm" H 3438 8625 50  0001 C CNN
 F 3 "" H 3400 8775 50  0001 C CNN
 	1    3400 8775

Commit message: Sensi board updated pin map
Parts:
- C16, C17, C18, C19, C2, C4, C5, C6: footprint Capacitor_SMD:C_0603_1608Metric -> Capacitor_SMD:C_0402_1005Metric
Changed lines of the file:
@@
 F 0 "C4" H 3765 1546 50  0000 L CNN
 F 1 "100n" H 3765 1455 50  0000 L CNN
-F 2 "Capacitor_SMD:C_0603_1608Metric" H 3688 1350 50  0001 C CNN
+F 2 "Capacitor_SMD:C_0402_1005Metric" H 3688 1350 50  0001 C CNN
 F 3 "" H 3650 1500 50  0001 C CNN
 	1    3650 1500
@@
 F 0 "C6" H 4215 1546 50  0000 L CNN
 F 1 "100n" H 4215 1455 50  0000 L CNN
-F 2 "Capacitor_SMD:C_0603_1608Metric" H 4138 1350 50  0001 C CNN
+F 2 "Capacitor_SMD:C_0402_1005Metric" H 4138 1350 50  0001 C CNN
 F 3 "" H 4100 1500 50  0001 C CNN
 	1    4100 1500
@@
 F 0 "C17" H 7590 1521 50  0000 L CNN
 F 1 "100n" H 7590 1430 50  0000 L CNN
-F 2 "Capacitor_SMD:C_0603_1608Metric" H 7513 1325 50  0001 C CNN
+F 2 "Capacitor_SMD:C_0402_1005Metric" H 7513 1325 50  0001 C CNN
 F 3 "" H 7475 1475 50  0001 C CNN
 	1    7475 1475
@@
 F 0 "C19" H 8040 1521 50  0000 L CNN
 F 1 "100n" H 8040 1430 50  0000 L CNN
-F 2 "Capacitor_SMD:C_0603_1608Metric" H 7963 1325 50  0001 C CNN
+F 2 "Capacitor_SMD:C_0402_1005Metric" H 7963 1325 50  0001 C CNN
 F 3 "" H 7925 1475 50  0001 C CNN
 	1    7925 1475
@@
 F 0 "C2" H 3765 6271 50  0000 L CNN
 F 1 "100n" H 3765 6180 50  0000 L CNN
-F 2 "Capacitor_SMD:C_0603_1608Metric" H 3688 6075 50  0001 C CNN
+F 2 "Capacitor_SMD:C_0402_1005Metric" H 3688 6075 50  0001 C CNN
 F 3 "" H 3650 6225 50  0001 C CNN
 	1    3650 6225
@@
 F 0 "C5" H 4215 6271 50  0000 L CNN
 F 1 "100n" H 4215 6180 50  0000 L CNN
-F 2 "Capacitor_SMD:C_0603_1608Metric" H 4138 6075 50  0001 C CNN
+F 2 "Capacitor_SMD:C_0402_1005Metric" H 4138 6075 50  0001 C CNN
 F 3 "" H 4100 6225 50  0001 C CNN
 	1    4100 6225
@@
 F 0 "C16" H 7565 6171 50  0000 L CNN
 F 1 "100n" H 7565 6080 50  0000 L CNN
-F 2 "Capacitor_SMD:C_0603_1608Metric" H 7488 5975 50  0001 C CNN
+F 2 "Capacitor_SMD:C_0402_1005Metric" H 7488 5975 50  0001 C CNN
 F 3 "" H 7450 6125 50  0001 C CNN
 	1    7450 6125
@@
 F 0 "C18" H 8015 6171 50  0000 L CNN
 F 1 "100n" H 8015 6080 50  0000 L CNN
-F 2 "Capacitor_SMD:C_0603_1608Metric" H 7938 5975 50  0001 C CNN
+F 2 "Capacitor_SMD:C_0402_1005Metric" H 7938 5975 50  0001 C CNN
 F 3 "" H 7900 6125 50  0001 C CNN
 	1    7900 6125

Commit message: Updated sensi board pin map and layout before PCB tracking
Parts:
- C1: footprint Crystal:Crystal_SMD_TXC_7A-2Pin_5x3.2mm -> Capacitor_SMD:C_0603_1608Metric; Devtank (none) -> 105-002
- C16, C17, C18, C19, C2, C4, C5, C6: Devtank (none) -> 105-019
- C3, C7, C8: Devtank (none) -> 105-002
- R1, R2, R5, R6: Devtank (none) -> 101-001
- R12, R3, R4, R7: Devtank (none) -> 101-010
- SW2, SW3, SW4, SW5: Devtank (none) -> 193-003
- U10, U11, U8, U9: Devtank (none) -> 155-006
Changed lines of the file:
@@
 F 2 "Package_DFN_QFN:TQFN-20-1EP_5x5mm_P0.65mm_EP3.1x3.1mm" H 3150 2800 60  0001 C CNN
 F 3 "" H 3150 2800 60  0001 C CNN
+F 4 "155-006" H 3400 2750 50  0001 C CNN "Devtank"
 	1    3400 2750
 	1    0    0    -1
@@
 F 2 "Capacitor_SMD:C_0402_1005Metric" H 3688 1350 50  0001 C CNN
 F 3 "" H 3650 1500 50  0001 C CNN
+F 4 "105-019" H 3650 1500 50  0001 C CNN "Devtank"
 	1    3650 1500
 	1    0    0    -1
@@
 F 2 "Capacitor_SMD:C_0402_1005Metric" H 4138 1350 50  0001 C CNN
 F 3 "" H 4100 1500 50  0001 C CNN
+F 4 "105-019" H 4100 1500 50  0001 C CNN "Devtank"
 	1    4100 1500
 	1    0    0    -1
@@
 F 2 "Resistor_SMD:R_0603_1608Metric" V 2180 2600 50  0001 C CNN
 F 3 "" H 2250 2600 50  0001 C CNN
+F 4 "101-001" H 2250 2600 50  0001 C CNN "Devtank"
 	1    2250 2600
 	1    0    0    -1
@@
 F 2 "Resistor_SMD:R_0603_1608Metric" V 4530 1500 50  0001 C CNN
 F 3 "" H 4600 1500 50  0001 C CNN
+F 4 "101-010" H 4600 1500 50  0001 C CNN "Devtank"
 	1    4600 1500
 	1    0    0    -1
@@
 F 2 "Capacitor_SMD:C_0603_1608Metric" H 3438 3900 50  0001 C CNN
 F 3 "" H 3400 4050 50  0001 C CNN
+F 4 "105-002" H 3400 4050 50  0001 C CNN "Devtank"
 	1    3400 4050
 	0    1    1    0
@@
 F 2 "Button_Switch_SMD:SW_DIP_SPSTx04_Slide_Copal_CHS-04B_W7.62mm_P1.27mm" H 3425 4650 50  0001 C CNN
 F 3 "" H 3425 4650 50  0001 C CNN
+F 4 "193-003" H 3425 4650 50  0001 C CNN "Devtank"
 	1    3425 4650
 	1    0    0    -1
@@
 F 2 "Package_DFN_QFN:TQFN-20-1EP_5x5mm_P0.65mm_EP3.1x3.1mm" H 6975 2775 60  0001 C CNN
 F 3 "" H 6975 2775 60  0001 C CNN
+F 4 "155-006" H 7225 2725 50  0001 C CNN "Devtank"
 	1    7225 2725
 	1    0    0    -1
@@
 F 2 "Capacitor_SMD:C_0402_1005Metric" H 7513 1325 50  0001 C CNN
 F 3 "" H 7475 1475 50  0001 C CNN
+F 4 "105-019" H 7475 1475 50  0001 C CNN "Devtank"
 	1    7475 1475
 	1    0    0    -1
@@
 F 2 "Capacitor_SMD:C_0402_1005Metric" H 7963 1325 50  0001 C CNN
 F 3 "" H 7925 1475 50  0001 C CNN
+F 4 "105-019" H 7925 1475 50  0001 C CNN "Devtank"
 	1    7925 1475
 	1    0    0    -1
@@
 F 2 "Resistor_SMD:R_0603_1608Metric" V 6005 2575 50  0001 C CNN
 F 3 "" H 6075 2575 50  0001 C CNN
+F 4 "101-001" H 6075 2575 50  0001 C CNN "Devtank"
 	1    6075 2575
 	1    0    0    -1
@@
 F 2 "Resistor_SMD:R_0603_1608Metric" V 8355 1475 50  0001 C CNN
 F 3 "" H 8425 1475 50  0001 C CNN
+F 4 "101-010" H 8425 1475 50  0001 C CNN "Devtank"
 	1    8425 1475
 	1    0    0    -1
@@
 F 2 "Capacitor_SMD:C_0603_1608Metric" H 7263 3875 50  0001 C CNN
 F 3 "" H 7225 4025 50  0001 C CNN
+F 4 "105-002" H 7225 4025 50  0001 C CNN "Devtank"
 	1    7225 4025
 	0    1    1    0
@@
 F 2 "Button_Switch_SMD:SW_DIP_SPSTx04_Slide_Copal_CHS-04B_W7.62mm_P1.27mm" H 7250 4625 50  0001 C CNN
 F 3 "" H 7250 4625 50  0001 C CNN
+F 4 "193-003" H 7250 4625 50  0001 C CNN "Devtank"
 	1    7250 4625
 	1    0    0    -1
@@
 F 2 "Package_DFN_QFN:TQFN-20-1EP_5x5mm_P0.65mm_EP3.1x3.1mm" H 3150 7525 60  0001 C CNN
 F 3 "" H 3150 7525 60  0001 C CNN
+F 4 "155-006" H 3400 7475 50  0001 C CNN "Devtank"
 	1    3400 7475
 	1    0    0    -1
@@
 F 2 "Capacitor_SMD:C_0402_1005Metric" H 3688 6075 50  0001 C CNN
 F 3 "" H 3650 6225 50  0001 C CNN
+F 4 "105-019" H 3650 6225 50  0001 C CNN "Devtank"
 	1    3650 6225
 	1    0    0    -1
@@
 F 2 "Capacitor_SMD:C_0402_1005Metric" H 4138 6075 50  0001 C CNN
 F 3 "" H 4100 6225 50  0001 C CNN
+F 4 "105-019" H 4100 6225 50  0001 C CNN "Devtank"
 	1    4100 6225
 	1    0    0    -1
@@
 F 2 "Resistor_SMD:R_0603_1608Metric" V 2180 7325 50  0001 C CNN
 F 3 "" H 2250 7325 50  0001 C CNN
+F 4 "101-001" H 2250 7325 50  0001 C CNN "Devtank"
 	1    2250 7325
 	1    0    0    -1
@@
 F 2 "Resistor_SMD:R_0603_1608Metric" V 4530 6225 50  0001 C CNN
 F 3 "" H 4600 6225 50  0001 C CNN
+F 4 "101-010" H 4600 6225 50  0001 C CNN "Devtank"
 	1    4600 6225
 	1    0    0    -1
@@
 F 0 "C1" V 3150 8825 50  0000 C CNN
 F 1 "100n" V 3239 8775 50  0000 C CNN
-F 2 "Crystal:Crystal_SMD_TXC_7A-2Pin_5x3.2mm" H 3438 8625 50  0001 C CNN
+F 2 "Capacitor_SMD:C_0603_1608Metric" H 3438 8625 50  0001 C CNN
 F 3 "" H 3400 8775 50  0001 C CNN
+F 4 "105-002" H 3400 8775 50  0001 C CNN "Devtank"
 	1    3400 8775
 	0    1    1    0
@@
 F 2 "Button_Switch_SMD:SW_DIP_SPSTx04_Slide_Copal_CHS-04B_W7.62mm_P1.27mm" H 3425 9375 50  0001 C CNN
 F 3 "" H 3425 9375 50  0001 C CNN
+F 4 "193-003" H 3425 9375 50  0001 C CNN "Devtank"
 	1    3425 9375
 	1    0    0    -1
@@
 F 2 "Package_DFN_QFN:TQFN-20-1EP_5x5mm_P0.65mm_EP3.1x3.1mm" H 6950 7425 60  0001 C CNN
 F 3 "" H 6950 7425 60  0001 C CNN
+F 4 "155-006" H 7200 7375 50  0001 C CNN "Devtank"
 	1    7200 7375
 	1    0    0    -1
@@
 F 2 "Capacitor_SMD:C_0402_1005Metric" H 7488 5975 50  0001 C CNN
 F 3 "" H 7450 6125 50  0001 C CNN
+F 4 "105-019" H 7450 6125 50  0001 C CNN "Devtank"
 	1    7450 6125
 	1    0    0    -1
@@
 F 2 "Capacitor_SMD:C_0402_1005Metric" H 7938 5975 50  0001 C CNN
 F 3 "" H 7900 6125 50  0001 C CNN
+F 4 "105-019" H 7900 6125 50  0001 C CNN "Devtank"
 	1    7900 6125
 	1    0    0    -1
@@
 F 2 "Resistor_SMD:R_0603_1608Metric" V 5980 7225 50  0001 C CNN
 F 3 "" H 6050 7225 50  0001 C CNN
+F 4 "101-001" H 6050 7225 50  0001 C CNN "Devtank"
 	1    6050 7225
 	1    0    0    -1
@@
 F 2 "Resistor_SMD:R_0603_1608Metric" V 8330 6125 50  0001 C CNN
 F 3 "" H 8400 6125 50  0001 C CNN
+F 4 "101-010" H 8400 6125 50  0001 C CNN "Devtank"
 	1    8400 6125
 	1    0    0    -1
@@
 F 2 "Capacitor_SMD:C_0603_1608Metric" H 7238 8525 50  0001 C CNN
 F 3 "" H 7200 8675 50  0001 C CNN
+F 4 "105-002" H 7200 8675 50  0001 C CNN "Devtank"
 	1    7200 8675
 	0    1    1    0
@@
 F 2 "Button_Switch_SMD:SW_DIP_SPSTx04_Slide_Copal_CHS-04B_W7.62mm_P1.27mm" H 7225 9275 50  0001 C CNN
 F 3 "" H 7225 9275 50  0001 C CNN
+F 4 "193-003" H 7225 9275 50  0001 C CNN "Devtank"
 	1    7225 9275
 	1    0    0    -1

Commit message: Sensi board with references visible and without stitching vias
Parts:
- C1, C16, C17, C18, C19, C2, C3, C4, C5, C6, C7, C8: value 100n -> 100nF
- R1, R2, R5, R6: value 470 -> 470R
- R12, R3, R4, R7: value 10k -> 10K
Changed lines of the file:
@@
 P 3650 1500
 F 0 "C4" H 3765 1546 50  0000 L CNN
-F 1 "100n" H 3765 1455 50  0000 L CNN
+F 1 "100nF" H 3765 1455 50  0000 L CNN
 F 2 "Capacitor_SMD:C_0402_1005Metric" H 3688 1350 50  0001 C CNN
 F 3 "" H 3650 1500 50  0001 C CNN
@@
 P 4100 1500
 F 0 "C6" H 4215 1546 50  0000 L CNN
-F 1 "100n" H 4215 1455 50  0000 L CNN
+F 1 "100nF" H 4215 1455 50  0000 L CNN
 F 2 "Capacitor_SMD:C_0402_1005Metric" H 4138 1350 50  0001 C CNN
 F 3 "" H 4100 1500 50  0001 C CNN
@@
 P 2250 2600
 F 0 "R2" H 2320 2646 50  0000 L CNN
-F 1 "470" H 2320 2555 50  0000 L CNN
+F 1 "470R" H 2320 2555 50  0000 L CNN
 F 2 "Resistor_SMD:R_0603_1608Metric" V 2180 2600 50  0001 C CNN
 F 3 "" H 2250 2600 50  0001 C CNN
@@
 P 4600 1500
 F 0 "R4" H 4670 1546 50  0000 L CNN
-F 1 "10k" H 4670 1455 50  0000 L CNN
+F 1 "10K" H 4670 1455 50  0000 L CNN
 F 2 "Resistor_SMD:R_0603_1608Metric" V 4530 1500 50  0001 C CNN
 F 3 "" H 4600 1500 50  0001 C CNN
@@
 P 3400 4050
 F 0 "C3" V 3150 4100 50  0000 C CNN
-F 1 "100n" V 3239 4050 50  0000 C CNN
+F 1 "100nF" V 3239 4050 50  0000 C CNN
 F 2 "Capacitor_SMD:C_0603_1608Metric" H 3438 3900 50  0001 C CNN
 F 3 "" H 3400 4050 50  0001 C CNN
@@
 P 7475 1475
 F 0 "C17" H 7590 1521 50  0000 L CNN
-F 1 "100n" H 7590 1430 50  0000 L CNN
+F 1 "100nF" H 7590 1430 50  0000 L CNN
 F 2 "Capacitor_SMD:C_0402_1005Metric" H 7513 1325 50  0001 C CNN
 F 3 "" H 7475 1475 50  0001 C CNN
@@
 P 7925 1475
 F 0 "C19" H 8040 1521 50  0000 L CNN
-F 1 "100n" H 8040 1430 50  0000 L CNN
+F 1 "100nF" H 8040 1430 50  0000 L CNN
 F 2 "Capacitor_SMD:C_0402_1005Metric" H 7963 1325 50  0001 C CNN
 F 3 "" H 7925 1475 50  0001 C CNN
@@
 P 6075 2575
 F 0 "R6" H 6145 2621 50  0000 L CNN
-F 1 "470" H 6145 2530 50  0000 L CNN
+F 1 "470R" H 6145 2530 50  0000 L CNN
 F 2 "Resistor_SMD:R_0603_1608Metric" V 6005 2575 50  0001 C CNN
 F 3 "" H 6075 2575 50  0001 C CNN
@@
 P 8425 1475
 F 0 "R12" H 8495 1521 50  0000 L CNN
-F 1 "10k" H 8495 1430 50  0000 L CNN
+F 1 "10K" H 8495 1430 50  0000 L CNN
 F 2 "Resistor_SMD:R_0603_1608Metric" V 8355 1475 50  0001 C CNN
 F 3 "" H 8425 1475 50  0001 C CNN
@@
 P 7225 4025
 F 0 "C8" V 6975 4075 50  0000 C CNN
-F 1 "100n" V 7064 4025 50  0000 C CNN
+F 1 "100nF" V 7064 4025 50  0000 C CNN
 F 2 "Capacitor_SMD:C_0603_1608Metric" H 7263 3875 50  0001 C CNN
 F 3 "" H 7225 4025 50  0001 C CNN
@@
 P 3650 6225
 F 0 "C2" H 3765 6271 50  0000 L CNN
-F 1 "100n" H 3765 6180 50  0000 L CNN
+F 1 "100nF" H 3765 6180 50  0000 L CNN
 F 2 "Capacitor_SMD:C_0402_1005Metric" H 3688 6075 50  0001 C CNN
 F 3 "" H 3650 6225 50  0001 C CNN
@@
 P 4100 6225
 F 0 "C5" H 4215 6271 50  0000 L CNN
-F 1 "100n" H 4215 6180 50  0000 L CNN
+F 1 "100nF" H 4215 6180 50  0000 L CNN
 F 2 "Capacitor_SMD:C_0402_1005Metric" H 4138 6075 50  0001 C CNN
 F 3 "" H 4100 6225 50  0001 C CNN
@@
 P 2250 7325
 F 0 "R1" H 2320 7371 50  0000 L CNN
-F 1 "470" H 2320 7280 50  0000 L CNN
+F 1 "470R" H 2320 7280 50  0000 L CNN
 F 2 "Resistor_SMD:R_0603_1608Metric" V 2180 7325 50  0001 C CNN
 F 3 "" H 2250 7325 50  0001 C CNN
@@
 P 4600 6225
 F 0 "R3" H 4670 6271 50  0000 L CNN
-F 1 "10k" H 4670 6180 50  0000 L CNN
+F 1 "10K" H 4670 6180 50  0000 L CNN
 F 2 "Resistor_SMD:R_0603_1608Metric" V 4530 6225 50  0001 C CNN
 F 3 "" H 4600 6225 50  0001 C CNN
@@
 P 3400 8775
 F 0 "C1" V 3150 8825 50  0000 C CNN
-F 1 "100n" V 3239 8775 50  0000 C CNN
+F 1 "100nF" V 3239 8775 50  0000 C CNN
 F 2 "Capacitor_SMD:C_0603_1608Metric" H 3438 8625 50  0001 C CNN
 F 3 "" H 3400 8775 50  0001 C CNN
@@
 P 7450 6125
 F 0 "C16" H 7565 6171 50  0000 L CNN
-F 1 "100n" H 7565 6080 50  0000 L CNN
+F 1 "100nF" H 7565 6080 50  0000 L CNN
 F 2 "Capacitor_SMD:C_0402_1005Metric" H 7488 5975 50  0001 C CNN
 F 3 "" H 7450 6125 50  0001 C CNN
@@
 P 7900 6125
 F 0 "C18" H 8015 6171 50  0000 L CNN
-F 1 "100n" H 8015 6080 50  0000 L CNN
+F 1 "100nF" H 8015 6080 50  0000 L CNN
 F 2 "Capacitor_SMD:C_0402_1005Metric" H 7938 5975 50  0001 C CNN
 F 3 "" H 7900 6125 50  0001 C CNN
@@
 P 6050 7225
 F 0 "R5" H 6120 7271 50  0000 L CNN
-F 1 "470" H 6120 7180 50  0000 L CNN
+F 1 "470R" H 6120 7180 50  0000 L CNN
 F 2 "Resistor_SMD:R_0603_1608Metric" V 5980 7225 50  0001 C CNN
 F 3 "" H 6050 7225 50  0001 C CNN
@@
 P 8400 6125
 F 0 "R7" H 8470 6171 50  0000 L CNN
-F 1 "10k" H 8470 6080 50  0000 L CNN
+F 1 "10K" H 8470 6080 50  0000 L CNN
 F 2 "Resistor_SMD:R_0603_1608Metric" V 8330 6125 50  0001 C CNN
 F 3 "" H 8400 6125 50  0001 C CNN
@@
 P 7200 8675
 F 0 "C7" V 6950 8725 50  0000 C CNN
-F 1 "100n" V 7039 8675 50  0000 C CNN
+F 1 "100nF" V 7039 8675 50  0000 C CNN
 F 2 "Capacitor_SMD:C_0603_1608Metric" H 7238 8525 50  0001 C CNN
 F 3 "" H 7200 8675 50  0001 C CNN
