File: kicad_hiltop_sensi_board/RelayOutputs.sch (KiCad schematic (older format))
At the start: 7 parts, among them K1 HRS1KH-S, Q2 ZXMN6A07F

Commit message: Just about to aad the RTD
Parts:
- D2: symbol device:LED -> Sensi_Board-rescue:LED-device
- D4: symbol device:D_Schottky -> Sensi_Board-rescue:D_Schottky-device
- K1: symbol Relay:G5Q-1 -> Sensi_Board-rescue:G5Q-1-Relay
- Q2: symbol device:Q_NMOS_GSD -> Sensi_Board-rescue:Q_NMOS_GSD-device
- R48, R50, R52: symbol device:R -> Sensi_Board-rescue:R-device
Changed lines of the file:
@@
 EESchema Schematic File Version 4
 LIBS:Sensi_Board-cache
-EELAYER 29 0
+EELAYER 30 0
 EELAYER END
 $Descr A3 16535 11693
 encoding utf-8
-Sheet 3 8
+Sheet 3 9
 Title "Iota Board"
 Date "2018-11-07"
@@
 $EndDescr
 $Comp
-L Relay:G5Q-1 K?
+L Sensi_Board-rescue:G5Q-1-Relay K?
 U 1 1 5BE5E5DE
 P 4200 2950
@@
 $EndComp
 $Comp
-L device:D_Schottky D?
+L Sensi_Board-rescue:D_Schottky-device D?
 U 1 1 5BE5E5E5
 P 3500 2800
@@
 $EndComp
 $Comp
-L device:Q_NMOS_GSD Q?
+L Sensi_Board-rescue:Q_NMOS_GSD-device Q?
 U 1 1 5BE5E5EC
 P 4100 3525
@@
 $EndComp
 $Comp
-L device:R R?
+L Sensi_Board-rescue:R-device R?
 U 1 1 5BE5E5F3
 P 3450 3525
@@
 $EndComp
 $Comp
-L device:R R?
+L Sensi_Board-rescue:R-device R?
 U 1 1 5BE5E5FA
 P 3800 3800
@@
 	4600 3225 5400 3225
 $Comp
-L device:LED D?
+L Sensi_Board-rescue:LED-device D?
 U 1 1 5BE5E626
 P 3025 2575
@@
 $EndComp
 $Comp
-L device:R R?
+L Sensi_Board-rescue:R-device R?
 U 1 1 5BE5E62D
 P 3025 2975
