File: kicad_hiltop_sensi_board/RelayOutputs.sch (KiCad schematic (older format))
At the start: 7 parts, among them K1 HRS1KH-S, Q2 ZXMN6A07F

Commit message: Sensi Board RevB
Connections:
- net +5V: now also D2.2 (A); no longer D2.1 (K)
- net at R48.2: now also D2.1 (K); no longer D2.2 (A)
Other:
- moved on the sheet: D2
Changed lines of the file:
@@
 F 4 "110-002" H 0   0   50  0001 C CNN "Devtank"
 	1    3025 2575
-	0    1    1    0
+	0    -1   -1   0
 $EndComp
 $Comp
