File: kicad_hiltop_sensi_board/Thermocouple inputs.sch (KiCad schematic (older format))
At the start: 52 parts, among them U21 MAX4194, U23 MAX4194, U24 MAX4194, U25 MAX4194

Commit message: Pressure sensor calcs added to 4-20mA circuit
Parts:
- C47, C49, C50, C54, C59, C65, C69, C71: Devtank 106-004 -> 105-026
Changed lines of the file:
@@
 EESchema Schematic File Version 4
 LIBS:Sensi_Board-cache
-EELAYER 29 0
+EELAYER 30 0
 EELAYER END
 $Descr A4 11693 8268
@@
 F 2 "Capacitor_SMD:C_0603_1608Metric" H 3438 2500 50  0001 C CNN
 F 3 "" H 3400 2650 50  0001 C CNN
-F 4 "106-004" H 3400 2650 50  0001 C CNN "Devtank"
+F 4 "105-026" H 3400 2650 50  0001 C CNN "Devtank"
 	1    3400 2650
 	1    0    0    -1
@@
 F 2 "Capacitor_SMD:C_0603_1608Metric" H 3438 1600 50  0001 C CNN
 F 3 "" H 3400 1750 50  0001 C CNN
-F 4 "106-004" H 3400 1750 50  0001 C CNN "Devtank"
+F 4 "105-026" H 3400 1750 50  0001 C CNN "Devtank"
 	1    3400 1750
 	1    0    0    -1
@@
 F 2 "Capacitor_SMD:C_0603_1608Metric" H 7658 2495 50  0001 C CNN
 F 3 "" H 7620 2645 50  0001 C CNN
-F 4 "106-004" H 7620 2645 50  0001 C CNN "Devtank"
+F 4 "105-026" H 7620 2645 50  0001 C CNN "Devtank"
 	1    7620 2645
 	1    0    0    -1
@@
 F 2 "Capacitor_SMD:C_0603_1608Metric" H 7658 1595 50  0001 C CNN
 F 3 "" H 7620 1745 50  0001 C CNN
-F 4 "106-004" H 7620 1745 50  0001 C CNN "Devtank"
+F 4 "105-026" H 7620 1745 50  0001 C CNN "Devtank"
 	1    7620 1745
 	1    0    0    -1
@@
 F 2 "Capacitor_SMD:C_0603_1608Metric" H 3433 5010 50  0001 C CNN
 F 3 "" H 3395 5160 50  0001 C CNN
-F 4 "106-004" H 3395 5160 50  0001 C CNN "Devtank"
+F 4 "105-026" H 3395 5160 50  0001 C CNN "Devtank"
 	1    3395 5160
 	1    0    0    -1
@@
 F 2 "Capacitor_SMD:C_0603_1608Metric" H 3433 4110 50  0001 C CNN
 F 3 "" H 3395 4260 50  0001 C CNN
-F 4 "106-004" H 3395 4260 50  0001 C CNN "Devtank"
+F 4 "105-026" H 3395 4260 50  0001 C CNN "Devtank"
 	1    3395 4260
 	1    0    0    -1
@@
 F 2 "Capacitor_SMD:C_0603_1608Metric" H 7648 5035 50  0001 C CNN
 F 3 "" H 7610 5185 50  0001 C CNN
-F 4 "106-004" H 7610 5185 50  0001 C CNN "Devtank"
+F 4 "105-026" H 7610 5185 50  0001 C CNN "Devtank"
 	1    7610 5185
 	1    0    0    -1
@@
 F 2 "Capacitor_SMD:C_0603_1608Metric" H 7648 4135 50  0001 C CNN
 F 3 "" H 7610 4285 50  0001 C CNN
-F 4 "106-004" H 7610 4285 50  0001 C CNN "Devtank"
+F 4 "105-026" H 7610 4285 50  0001 C CNN "Devtank"
 	1    7610 4285
 	1    0    0    -1
