File: kicad_hiltop_sensi_board/Thermocouple inputs.sch (KiCad schematic (older format))
At the start: 52 parts, among them U21 MAX4194, U23 MAX4194, U24 MAX4194, U25 MAX4194

Commit message: updated footprints to simplify bom
Parts:
- C53, C68, C72, C83: value 0.1uF -> 100nF
Changed lines of the file:
@@
 P 5075 1800
 F 0 "C68" V 4823 1800 50  0000 C CNN
-F 1 "0.1uF" V 4914 1800 50  0000 C CNN
+F 1 "100nF" V 4914 1800 50  0000 C CNN
 F 2 "Capacitor_SMD:C_0402_1005Metric" H 5113 1650 50  0001 C CNN
 F 3 "" H 5075 1800 50  0001 C CNN
@@
 P 9295 1795
 F 0 "C83" V 9043 1795 50  0000 C CNN
-F 1 "0.1uF" V 9134 1795 50  0000 C CNN
+F 1 "100nF" V 9134 1795 50  0000 C CNN
 F 2 "Capacitor_SMD:C_0402_1005Metric" H 9333 1645 50  0001 C CNN
 F 3 "" H 9295 1795 50  0001 C CNN
@@
 P 5070 4310
 F 0 "C53" V 4818 4310 50  0000 C CNN
-F 1 "0.1uF" V 4909 4310 50  0000 C CNN
+F 1 "100nF" V 4909 4310 50  0000 C CNN
 F 2 "Capacitor_SMD:C_0402_1005Metric" H 5108 4160 50  0001 C CNN
 F 3 "" H 5070 4310 50  0001 C CNN
@@
 P 9285 4335
 F 0 "C72" V 9033 4335 50  0000 C CNN
-F 1 "0.1uF" V 9124 4335 50  0000 C CNN
+F 1 "100nF" V 9124 4335 50  0000 C CNN
 F 2 "Capacitor_SMD:C_0402_1005Metric" H 9323 4185 50  0001 C CNN
 F 3 "" H 9285 4335 50  0001 C CNN
