File: kicad_hiltop_sensi_board/USB2502 Hub Controller.sch (KiCad schematic (older format))
At the start: 49 parts, among them U27 USB2502, U7 DNF, Y1 50ppm 24.000MHZ

Commit message: Sensi Board Complete
Parts:
- C100, C102, C103, C104, C105: Devtank 105-025 -> 105-028
- C106: Devtank 105-019 -> (none)
- D3, D5: Devtank (none) -> 110-002
- L1: Devtank (none) -> 113-004
- R112: Devtank 101-010 -> (none)
- R121, R66: Devtank (none) -> 101-005
- R137, R138, R143, R144: value DNP -> DNF
- R139, R140: Devtank (none) -> 101-015
- R141, R142: Devtank (none) -> 101-024
- U7: Devtank 129-006 -> (none)
Changed lines of the file:
@@
 F 4 "6.3V" H 8400 7200 50  0001 C CNN "Voltage"
 F 5 "X5R" H 8400 7200 50  0001 C CNN "Dielectric"
-F 6 "105-025" H 8400 7200 50  0001 C CNN "Devtank"
+F 6 "105-028" H 8400 7200 50  0001 C CNN "Devtank"
 	1    8400 7200
 	1    0    0    -1
@@
 F 4 "6.3V" H 8000 7650 50  0001 C CNN "Voltage"
 F 5 "X5R" H 8000 7650 50  0001 C CNN "Dielectric"
-F 6 "105-025" H 8000 7650 50  0001 C CNN "Devtank"
+F 6 "105-028" H 8000 7650 50  0001 C CNN "Devtank"
 	1    8000 7650
 	1    0    0    -1
@@
 F 4 "6.3V" H 8000 6750 50  0001 C CNN "Voltage"
 F 5 "X5R" H 8000 6750 50  0001 C CNN "Dielectric"
-F 6 "105-025" H 8000 6750 50  0001 C CNN "Devtank"
+F 6 "105-028" H 8000 6750 50  0001 C CNN "Devtank"
 	1    8000 6750
 	1    0    0    -1
@@
 F 4 "6.3V" H 8400 6250 50  0001 C CNN "Voltage"
 F 5 "X5R" H 8400 6250 50  0001 C CNN "Dielectric"
-F 6 "105-025" H 8400 6250 50  0001 C CNN "Devtank"
+F 6 "105-028" H 8400 6250 50  0001 C CNN "Devtank"
 	1    8400 6250
 	1    0    0    -1
@@
 F 2 "Capacitor_SMD:C_0402_1005Metric" H 9938 5600 50  0001 C CNN
 F 3 "" H 9900 5750 50  0001 C CNN
-F 4 "105-019" H 9900 5750 50  0001 C CNN "Devtank"
+F 4 "" H 9900 5750 50  0001 C CNN "Devtank"
 	1    9900 5750
 	1    0    0    -1
@@
 F 2 "Resistor_SMD:R_0603_1608Metric" V 9830 5350 50  0001 C CNN
 F 3 "" H 9900 5350 50  0001 C CNN
-F 4 "101-010" H 9900 5350 50  0001 C CNN "Devtank"
+F 4 "" H 9900 5350 50  0001 C CNN "Devtank"
 	1    9900 5350
 	1    0    0    -1
@@
 F 4 "6.3V" H 8000 8100 50  0001 C CNN "Voltage"
 F 5 "X5R" H 8000 8100 50  0001 C CNN "Dielectric"
-F 6 "105-025" H 8000 8100 50  0001 C CNN "Devtank"
+F 6 "105-028" H 8000 8100 50  0001 C CNN "Devtank"
 	1    8000 8100
 	1    0    0    -1
@@
 F 2 "Inductor_SMD:L_0805_2012Metric" V 7680 8700 50  0001 C CNN
 F 3 "" H 7750 8700 50  0001 C CNN
+F 4 "113-004" H 7750 8700 50  0001 C CNN "Devtank"
 	1    7750 8700
 	0    1    1    0
@@
 F 2 "Package_SO:SOIC-8_3.9x4.9mm_P1.27mm" H 9300 5150 60  0001 C CNN
 F 3 "" H 9300 5150 60  0001 C CNN
-F 4 "129-006" H 9350 5700 50  0001 C CNN "Devtank"
+F 4 "" H 9350 5700 50  0001 C CNN "Devtank"
 	1    9350 5700
 	1    0    0    -1
@@
 P 10215 4365
 F 0 "R143" V 10422 4365 50  0000 C CNN
-F 1 "DNP" V 10331 4365 50  0000 C CNN
+F 1 "DNF" V 10331 4365 50  0000 C CNN
 F 2 "Resistor_SMD:R_0603_1608Metric" V 10145 4365 50  0001 C CNN
 F 3 "" H 10215 4365 50  0001 C CNN
@@
 F 2 "Resistor_SMD:R_0603_1608Metric" V 9695 4365 50  0001 C CNN
 F 3 "" H 9765 4365 50  0001 C CNN
+F 4 "101-024" H 9765 4365 50  0001 C CNN "Devtank"
 	1    9765 4365
 	0    -1   -1   0
@@
 P 9315 4365
 F 0 "R137" V 9522 4365 50  0000 C CNN
-F 1 "DNP" V 9431 4365 50  0000 C CNN
+F 1 "DNF" V 9431 4365 50  0000 C CNN
 F 2 "Resistor_SMD:R_0603_1608Metric" V 9245 4365 50  0001 C CNN
 F 3 "" H 9315 4365 50  0001 C CNN
@@
 F 2 "Resistor_SMD:R_0603_1608Metric" V 8820 4365 50  0001 C CNN
 F 3 "" H 8890 4365 50  0001 C CNN
+F 4 "101-005" H 8890 4365 50  0001 C CNN "Devtank"
 	1    8890 4365
 	0    -1   -1   0
@@
 F 2 "Resistor_SMD:R_0603_1608Metric" V 9470 4570 50  0001 C CNN
 F 3 "" H 9540 4570 50  0001 C CNN
+F 4 "101-015" H 9540 4570 50  0001 C CNN "Devtank"
 	1    9540 4570
 	0    -1   -1   0
@@
 F 2 "LED_SMD:LED_0603_1608Metric" H 9540 4825 50  0001 C CNN
 F 3 "~" H 9540 4825 50  0001 C CNN
+F 4 "110-002" H 9540 4825 50  0001 C CNN "Devtank"
 	1    9540 4825
 	1    0    0    -1
@@
 P 10220 3505
 F 0 "R144" V 10427 3505 50  0000 C CNN
-F 1 "DNP" V 10336 3505 50  0000 C CNN
+F 1 "DNF" V 10336 3505 50  0000 C CNN
 F 2 "Resistor_SMD:R_0603_1608Metric" V 10150 3505 50  0001 C CNN
 F 3 "" H 10220 3505 50  0001 C CNN
@@
 F 2 "Resistor_SMD:R_0603_1608Metric" V 9700 3505 50  0001 C CNN
 F 3 "" H 9770 3505 50  0001 C CNN
+F 4 "101-024" H 9770 3505 50  0001 C CNN "Devtank"
 	1    9770 3505
 	0    -1   -1   0
@@
 P 9320 3505
 F 0 "R138" V 9527 3505 50  0000 C CNN
-F 1 "DNP" V 9436 3505 50  0000 C CNN
+F 1 "DNF" V 9436 3505 50  0000 C CNN
 F 2 "Resistor_SMD:R_0603_1608Metric" V 9250 3505 50  0001 C CNN
 F 3 "" H 9320 3505 50  0001 C CNN
@@
 F 2 "Resistor_SMD:R_0603_1608Metric" V 8825 3505 50  0001 C CNN
 F 3 "" H 8895 3505 50  0001 C CNN
+F 4 "101-005" H 8895 3505 50  0001 C CNN "Devtank"
 	1    8895 3505
 	0    -1   -1   0
@@
 F 2 "Resistor_SMD:R_0603_1608Metric" V 9475 3715 50  0001 C CNN
 F 3 "" H 9545 3715 50  0001 C CNN
+F 4 "101-015" H 9545 3715 50  0001 C CNN "Devtank"
 	1    9545 3715
 	0    -1   -1   0
@@
 F 2 "LED_SMD:LED_0603_1608Metric" H 9545 3965 50  0001 C CNN
 F 3 "~" H 9545 3965 50  0001 C CNN
+F 4 "110-002" H 9545 3965 50  0001 C CNN "Devtank"
 	1    9545 3965
 	1    0    0    -1

Commit message: Pressure sensor calcs added to 4-20mA circuit
Parts:
- C91: Devtank 105-026 -> 105-025
- Y1: Devtank 181-010 -> 181-011
Changed lines of the file:
@@
 EESchema Schematic File Version 4
 LIBS:Sensi_Board-cache
-EELAYER 29 0
+EELAYER 30 0
 EELAYER END
 $Descr A3 16535 11693
@@
 F 2 "Crystal:Crystal_SMD_TXC_7A-2Pin_5x3.2mm" H 4150 8550 50  0001 C CNN
 F 3 "" H 4150 8550 50  0001 C CNN
-F 4 "181-010" H 4150 8550 50  0001 C CNN "Devtank"
+F 4 "181-011" H 4150 8550 50  0001 C CNN "Devtank"
 	1    4150 8550
 	0    -1   -1   0
@@
 F 4 "16V" H 5250 2200 50  0001 C CNN "Voltage"
 F 5 "X5R" H 5250 2200 50  0001 C CNN "Dielectric"
-F 6 "105-026" H 5250 2200 50  0001 C CNN "Devtank"
+F 6 "105-025" H 5250 2200 50  0001 C CNN "Devtank"
 	1    5250 2200
 	1    0    0    -1
